File: hardware/breakout_boards/stm32l151_breakout/_saved_stm32l151_breakout.sch (KiCad schematic (older format))
At the start: 14 parts, among them J1 USB_B_Micro, J2 Conn_01x24_Male, J3 Conn_ARM_JTAG_SWD_10, J4 Conn_01x24_Male, U1 LD1117-3.3, U2 STM32L151C

Commit message: Finish out initial board
Parts:
- D1: footprint (none) -> LEDs:LED_0805_HandSoldering
- R1: value R -> 40; footprint (none) -> Resistors_SMD:R_0805_HandSoldering
Changed lines of the file:
@@
 F 0 "D1" V 2688 6583 50  0000 R CNN
 F 1 "LED" V 2597 6583 50  0000 R CNN
-F 2 "" H 2650 6700 50  0001 C CNN
+F 2 "LEDs:LED_0805_HandSoldering" H 2650 6700 50  0001 C CNN
 F 3 "~" H 2650 6700 50  0001 C CNN
 	1    2650 6700
@@
 Connection ~ 2650 6350
 $Comp
-L power:GND #PWR?
+L power:GND #PWR012
 U 1 1 5A33D07D
 P 2650 7250
-F 0 "#PWR?" H 2650 7000 50  0001 C CNN
+F 0 "#PWR012" H 2650 7000 50  0001 C CNN
 F 1 "GND" H 2655 7077 50  0000 C CNN
 F 2 "" H 2650 7250 50  0001 C CNN
@@
 P 2650 7050
 F 0 "R1" H 2720 7096 50  0000 L CNN
-F 1 "R" H 2720 7005 50  0000 L CNN
-F 2 "" V 2580 7050 50  0001 C CNN
+F 1 "40" H 2720 7005 50  0000 L CNN
+F 2 "Resistors_SMD:R_0805_HandSoldering" V 2580 7050 50  0001 C CNN
 F 3 "" H 2650 7050 50  0001 C CNN
 	1    2650 7050
