File: hardware/breakout_boards/stm32l151_breakout/stm32l151_raw_breakout/stm32l151_raw_breakout.sch (KiCad schematic (older format))
At the start: 49 parts, among them J1 Conn_01x01, J10 Conn_01x01, J11 Conn_01x01, J12 Conn_01x01, J13 Conn_01x01, J14 Conn_01x01, J15 Conn_01x01, J16 Conn_01x01, J17 Conn_01x01, J18 Conn_01x01, J19 Conn_01x01, J2 Conn_01x01, J20 Conn_01x01, J21 Conn_01x01, J22 Conn_01x01, J23 Conn_01x01, J24 Conn_01x01, J25 Conn_01x01, J26 Conn_01x01, J27 Conn_01x01, J28 Conn_01x01, J29 Conn_01x01, J3 Conn_01x01, J30 Conn_01x01, J31 Conn_01x01, J32 Conn_01x01, J33 Conn_01x01, J34 Conn_01x01, J35 Conn_01x01, J36 Conn_01x01, J37 Conn_01x01, J38 Conn_01x01, J39 Conn_01x01, J4 Conn_01x01, J40 Conn_01x01, J41 Conn_01x01, J42 Conn_01x01, J43 Conn_01x01, J44 Conn_01x01, J45 Conn_01x01, J46 Conn_01x01, J47 Conn_01x01, J48 Conn_01x01, J5 Conn_01x01, J6 Conn_01x01, J7 Conn_01x01, J8 Conn_01x01, J9 Conn_01x01, U1 STM32L151CCTx

Commit message: Diagonal STM32 raw breakout board
Parts:
- J1, J10, J11, J12, J13, J14, J15, J16, J17, J18, J19, J2, J20, J21, J22, J23, J24, J25, J26, J27, J28, J29, J3, J30, J31, J32, J33, J34, J35, J36, J37, J38, J39, J4, J40, J41, J42, J43, J44, J45, J46, J47, J48, J5, J6, J7, J8, J9: footprint (none) -> Pin_Headers:Pin_Header_Straight_1x01_Pitch1.27mm

Commit message: Save stm32 raw breakout board
Parts:
- J1, J10, J11, J12, J13, J14, J15, J16, J17, J18, J19, J2, J20, J21, J22, J23, J24, J25, J26, J27, J28, J29, J3, J30, J31, J32, J33, J34, J35, J36, J37, J38, J39, J4, J40, J41, J42, J43, J44, J45, J46, J47, J48, J5, J6, J7, J8, J9: symbol Connector:Conn_01x01 -> stm32l151_raw_breakout-rescue:Conn_01x01-Connector
Changed lines of the file:
@@
 $EndComp
 $Comp
-L Connector:Conn_01x01 J1
+L stm32l151_raw_breakout-rescue:Conn_01x01-Connector J1
 U 1 1 5AC94755
 P 800 2250
@@
 	1000 2250 1600 2250
 $Comp
-L Connector:Conn_01x01 J2
+L stm32l151_raw_breakout-rescue:Conn_01x01-Connector J2
 U 1 1 5AC947D9
 P 800 2450
@@
 	1000 2450 1600 2450
 $Comp
-L Connector:Conn_01x01 J3
+L stm32l151_raw_breakout-rescue:Conn_01x01-Connector J3
 U 1 1 5AC94826
 P 800 2650
@@
 	1000 2650 1600 2650
 $Comp
-L Connector:Conn_01x01 J4
+L stm32l151_raw_breakout-rescue:Conn_01x01-Connector J4
 U 1 1 5AC94897
 P 800 2850
@@
 	1000 2850 1600 2850
 $Comp
-L Connector:Conn_01x01 J5
+L stm32l151_raw_breakout-rescue:Conn_01x01-Connector J5
 U 1 1 5AC948FB
 P 800 2950
@@
 	1000 2950 1600 2950
 $Comp
-L Connector:Conn_01x01 J6
+L stm32l151_raw_breakout-rescue:Conn_01x01-Connector J6
 U 1 1 5AC94975
 P 800 3150
@@
 	1000 3150 1600 3150
 $Comp
-L Connector:Conn_01x01 J7
+L stm32l151_raw_breakout-rescue:Conn_01x01-Connector J7
 U 1 1 5AC94A00
 P 800 3250
@@
 	1000 3250 1600 3250
 $Comp
-L Connector:Conn_01x01 J8
+L stm32l151_raw_breakout-rescue:Conn_01x01-Connector J8
 U 1 1 5AC94AB5
 P 800 3350
@@
 	1000 3350 1600 3350
 $Comp
-L Connector:Conn_01x01 J9
+L stm32l151_raw_breakout-rescue:Conn_01x01-Connector J9
 U 1 1 5AC94B7C
 P 800 3550
@@
 $EndComp
 $Comp
-L Connector:Conn_01x01 J10
+L stm32l151_raw_breakout-rescue:Conn_01x01-Connector J10
 U 1 1 5AC94BEA
 P 800 3650
@@
 $EndComp
 $Comp
-L Connector:Conn_01x01 J11
+L stm32l151_raw_breakout-rescue:Conn_01x01-Connector J11
 U 1 1 5AC94C59
 P 800 3750
@@
 $EndComp
 $Comp
-L Connector:Conn_01x01 J12
+L stm32l151_raw_breakout-rescue:Conn_01x01-Connector J12
 U 1 1 5AC94CC9
 P 800 3850
@@
 $EndComp
 $Comp
-L Connector:Conn_01x01 J13
+L stm32l151_raw_breakout-rescue:Conn_01x01-Connector J13
 U 1 1 5AC94D3C
 P 800 3950
@@
 $EndComp
 $Comp
-L Connector:Conn_01x01 J14
+L stm32l151_raw_breakout-rescue:Conn_01x01-Connector J14
 U 1 1 5AC94DB6
 P 800 4050
@@
 $EndComp
 $Comp
-L Connector:Conn_01x01 J15
+L stm32l151_raw_breakout-rescue:Conn_01x01-Connector J15
 U 1 1 5AC94E33
 P 800 4150
@@
 $EndComp
 $Comp
-L Connector:Conn_01x01 J16
+L stm32l151_raw_breakout-rescue:Conn_01x01-Connector J16
 U 1 1 5AC94EB7
 P 800 4250
@@
 $EndComp
 $Comp
-L Connector:Conn_01x01 J17
+L stm32l151_raw_breakout-rescue:Conn_01x01-Connector J17
 U 1 1 5AC94F40
 P 800 4350
@@
 $EndComp
 $Comp
-L Connector:Conn_01x01 J18
+L stm32l151_raw_breakout-rescue:Conn_01x01-Connector J18
 U 1 1 5AC94FCE
 P 800 4450
@@
 $EndComp
 $Comp
-L Connector:Conn_01x01 J19
+L stm32l151_raw_breakout-rescue:Conn_01x01-Connector J19
 U 1 1 5AC95097
 P 800 4550
@@
 $EndComp
 $Comp
-L Connector:Conn_01x01 J20
+L stm32l151_raw_breakout-rescue:Conn_01x01-Connector J20
 U 1 1 5AC951CD
 P 800 4650
@@
 $EndComp
 $Comp
-L Connector:Conn_01x01 J21
+L stm32l151_raw_breakout-rescue:Conn_01x01-Connector J21
 U 1 1 5AC9526A
 P 800 4750
@@
 $EndComp
 $Comp
-L Connector:Conn_01x01 J22
+L stm32l151_raw_breakout-rescue:Conn_01x01-Connector J22
 U 1 1 5AC95312
 P 800 4850
@@
 $EndComp
 $Comp
-L Connector:Conn_01x01 J23
+L stm32l151_raw_breakout-rescue:Conn_01x01-Connector J23
 U 1 1 5AC953B7
 P 800 4950
@@
 $EndComp
 $Comp
-L Connector:Conn_01x01 J24
+L stm32l151_raw_breakout-rescue:Conn_01x01-Connector J24
 U 1 1 5AC95461
 P 800 5050
@@
 $EndComp
 $Comp
-L Connector:Conn_01x01 J25
+L stm32l151_raw_breakout-rescue:Conn_01x01-Connector J25
 U 1 1 5AC956D2
 P 5500 1250
@@
 $EndComp
 $Comp
-L Connector:Conn_01x01 J27
+L stm32l151_raw_breakout-rescue:Conn_01x01-Connector J27
 U 1 1 5AC95805
 P 5600 1250
@@
 $EndComp
 $Comp
-L Connector:Conn_01x01 J29
+L stm32l151_raw_breakout-rescue:Conn_01x01-Connector J29
 U 1 1 5AC958E4
 P 5700 1250
@@
 $EndComp
 $Comp
-L Connector:Conn_01x01 J31
+L stm32l151_raw_breakout-rescue:Conn_01x01-Connector J31
 U 1 1 5AC959C7
 P 5800 1250
@@
 $EndComp
 $Comp
-L Connector:Conn_01x01 J26
+L stm32l151_raw_breakout-rescue:Conn_01x01-Connector J26
 U 1 1 5AC95D38
 P 5500 6000
@@
 $EndComp
 $Comp
-L Connector:Conn_01x01 J28
+L stm32l151_raw_breakout-rescue:Conn_01x01-Connector J28
 U 1 1 5AC95F01
 P 5600 6000
@@
 $EndComp
 $Comp
-L Connector:Conn_01x01 J30
+L stm32l151_raw_breakout-rescue:Conn_01x01-Connector J30
 U 1 1 5AC9603E
 P 5700 6000
@@
 $EndComp
 $Comp
-L Connector:Conn_01x01 J32
+L stm32l151_raw_breakout-rescue:Conn_01x01-Connector J32
 U 1 1 5AC96181
 P 5800 6000
@@
 $EndComp
 $Comp
-L Connector:Conn_01x01 J33
+L stm32l151_raw_breakout-rescue:Conn_01x01-Connector J33
 U 1 1 5AC9643B
 P 10250 3550
@@
 $EndComp
 $Comp
-L Connector:Conn_01x01 J34
+L stm32l151_raw_breakout-rescue:Conn_01x01-Connector J34
 U 1 1 5AC964CB
 P 10250 3650
@@
 $EndComp
 $Comp
-L Connector:Conn_01x01 J35
+L stm32l151_raw_breakout-rescue:Conn_01x01-Connector J35
 U 1 1 5AC9655C
 P 10250 3750
@@
 $EndComp
 $Comp
-L Connector:Conn_01x01 J36
+L stm32l151_raw_breakout-rescue:Conn_01x01-Connector J36
 U 1 1 5AC965F0
 P 10250 3850
@@
 $EndComp
 $Comp
-L Connector:Conn_01x01 J37
+L stm32l151_raw_breakout-rescue:Conn_01x01-Connector J37
 U 1 1 5AC96687
 P 10250 3950
@@
 $EndComp
 $Comp
-L Connector:Conn_01x01 J38
+L stm32l151_raw_breakout-rescue:Conn_01x01-Connector J38
 U 1 1 5AC9677B
 P 10250 4050
@@
 $EndComp
 $Comp
-L Connector:Conn_01x01 J39
+L stm32l151_raw_breakout-rescue:Conn_01x01-Connector J39
 U 1 1 5AC96818
 P 10250 4150
@@
 $EndComp
 $Comp
-L Connector:Conn_01x01 J40
+L stm32l151_raw_breakout-rescue:Conn_01x01-Connector J40
 U 1 1 5AC968B8
 P 10250 4250
@@
 $EndComp
 $Comp
-L Connector:Conn_01x01 J41
+L stm32l151_raw_breakout-rescue:Conn_01x01-Connector J41
 U 1 1 5AC9695B
 P 10250 4350
@@
 $EndComp
 $Comp
-L Connector:Conn_01x01 J42
+L stm32l151_raw_breakout-rescue:Conn_01x01-Connector J42
 U 1 1 5AC96A55
 P 10250 4450
@@
 $EndComp
 $Comp
-L Connector:Conn_01x01 J43
+L stm32l151_raw_breakout-rescue:Conn_01x01-Connector J43
 U 1 1 5AC96AFE
 P 10250 4550
@@
 $EndComp
 $Comp
-L Connector:Conn_01x01 J44
+L stm32l151_raw_breakout-rescue:Conn_01x01-Connector J44
 U 1 1 5AC96BAA
 P 10250 4650
@@
 $EndComp
 $Comp
-L Connector:Conn_01x01 J45
+L stm32l151_raw_breakout-rescue:Conn_01x01-Connector J45
 U 1 1 5AC96C59
 P 10250 4750
@@
 $EndComp
 $Comp
-L Connector:Conn_01x01 J46
+L stm32l151_raw_breakout-rescue:Conn_01x01-Connector J46
 U 1 1 5AC96D0B
 P 10250 4850
@@
 $EndComp
 $Comp
-L Connector:Conn_01x01 J47
+L stm32l151_raw_breakout-rescue:Conn_01x01-Connector J47
 U 1 1 5AC96DC0
 P 10250 4950
@@
 $EndComp
 $Comp
-L Connector:Conn_01x01 J48
+L stm32l151_raw_breakout-rescue:Conn_01x01-Connector J48
 U 1 1 5AC96F84
 P 10250 5050
