File: hardware/breakout_boards/cs43l22_breakout/cs43l22_breakout.sch (KiCad schematic (older format))
At the start: 43 parts, among them J1 MCLK, J10 SPKR_OUTB+, J11 SPKR_OUTB-, J12 AIN1A, J13 AIN1B, J14 AIN2A, J15 AIN2B, J16 AIN3A, J17 AIN3B, J18 AIN4A, J19 AIN4B, J2 SCLK, J20 SJ-3524, J3 LRCK, J4 SDIN, J5 ~RESET, J6 SCL, J7 SDA, J8 SPKR_OUTA+, J9 SPKR_OUTA-, U1 CS43L22_V2

Commit message: Finish out cs43l22 breakout schematic
Parts:
- removed R5: 47, symbol Device:R_Small
- added U2: LM1117-1.8, TO_SOT_Packages_SMD:SOT-223, symbol Regulator_Linear:LM1117-1.8
- C1, C11, C12, C13, C14, C15, C16, C17, C2, C3, C4, C5, C6, C7, C8, C9: footprint (none) -> Capacitors_SMD:C_0805_HandSoldering
- C10: value C_Small -> 1uf; footprint (none) -> Capacitors_SMD:C_0805_HandSoldering
- J1, J10, J11, J12, J13, J14, J15, J16, J17, J18, J19, J2, J3, J4, J5, J6, J7, J8, J9: footprint (none) -> connector:Conn_1pin_2.54mm
- J20: footprint (none) -> audio:SJ-3524-SMT_Stereo_Jack
- R1, R2, R3, R4: footprint (none) -> Resistors_SMD:R_0805_HandSoldering
- U1: footprint (none) -> Housings_DFN_QFN:QFN-40-1EP_6x6mm_Pitch0.5mm
Connections:
- net labels added: +5V
- wire segments 95 -> 92

Commit message: Start spreading out the pcb
Parts:
- renumbered J12 to AIN1A1, J13 to AIN1B1, J14 to AIN2A1, J15 to AIN2B1, J16 to AIN3A1, J17 to AIN3B1, J18 to AIN4A1, J19 to AIN4B1, J3 to LRCK1, J1 to MCLK1, J6 to SCL1, J2 to SCLK1, J7 to SDA1, J4 to SDIN1, J8 to SPKR_OUTA+1, J9 to SPKR_OUTA-1, J10 to SPKR_OUTB+1, J11 to SPKR_OUTB-1, J5 to ~RESET1
Changed lines of the file:
@@
 	5800 3100 7450 3100
 $Comp
-L Connector:Conn_01x01_Male J8
+L Connector:Conn_01x01_Male SPKR_OUTA+1
 U 1 1 5AE73C2F
 P 7650 3000
-F 0 "J8" H 7622 2930 50  0000 R CNN
+F 0 "SPKR_OUTA+1" H 7622 2930 50  0000 R CNN
 F 1 "SPKR_OUTA+" H 7622 3021 50  0000 R CNN
 F 2 "connector:Conn_1pin_2.54mm" H 7650 3000 50  0001 C CNN
@@
 $EndComp
 $Comp
-L Connector:Conn_01x01_Male J9
+L Connector:Conn_01x01_Male SPKR_OUTA-1
 U 1 1 5AE73CD6
 P 7650 3100
-F 0 "J9" H 7600 3200 50  0000 R CNN
+F 0 "SPKR_OUTA-1" H 7600 3200 50  0000 R CNN
 F 1 "SPKR_OUTA-" H 7622 3121 50  0000 R CNN
 F 2 "connector:Conn_1pin_2.54mm" H 7650 3100 50  0001 C CNN
@@
 $EndComp
 $Comp
-L Connector:Conn_01x01_Male J10
+L Connector:Conn_01x01_Male SPKR_OUTB+1
 U 1 1 5AE73E30
 P 7650 3450
-F 0 "J10" H 7050 3450 50  0000 R CNN
+F 0 "SPKR_OUTB+1" H 7050 3450 50  0000 R CNN
 F 1 "SPKR_OUTB+" H 7623 3471 50  0000 R CNN
 F 2 "connector:Conn_1pin_2.54mm" H 7650 3450 50  0001 C CNN
@@
 $EndComp
 $Comp
-L Connector:Conn_01x01_Male J11
+L Connector:Conn_01x01_Male SPKR_OUTB-1
 U 1 1 5AE73E37
 P 7650 3550
-F 0 "J11" H 7050 3550 50  0000 R CNN
+F 0 "SPKR_OUTB-1" H 7050 3550 50  0000 R CNN
 F 1 "SPKR_OUTB-" H 7622 3571 50  0000 R CNN
 F 2 "connector:Conn_1pin_2.54mm" H 7650 3550 50  0001 C CNN
@@
 	5800 5100 7450 5100
 $Comp
-L Connector:Conn_01x01_Male J12
+L Connector:Conn_01x01_Male AIN1A1
 U 1 1 5AE76F8B
 P 7650 3700
-F 0 "J12" H 7350 3700 50  0000 R CNN
+F 0 "AIN1A1" H 7350 3700 50  0000 R CNN
 F 1 "AIN1A" H 7623 3721 50  0000 R CNN
 F 2 "connector:Conn_1pin_2.54mm" H 7650 3700 50  0001 C CNN
@@
 $EndComp
 $Comp
-L Connector:Conn_01x01_Male J13
+L Connector:Conn_01x01_Male AIN1B1
 U 1 1 5AE77184
 P 7650 3900
-F 0 "J13" H 7350 3900 50  0000 R CNN
+F 0 "AIN1B1" H 7350 3900 50  0000 R CNN
 F 1 "AIN1B" H 7623 3921 50  0000 R CNN
 F 2 "connector:Conn_1pin_2.54mm" H 7650 3900 50  0001 C CNN
@@
 $EndComp
 $Comp
-L Connector:Conn_01x01_Male J14
+L Connector:Conn_01x01_Male AIN2A1
 U 1 1 5AE777D1
 P 7650 4100
-F 0 "J14" H 7350 4100 50  0000 R CNN
+F 0 "AIN2A1" H 7350 4100 50  0000 R CNN
 F 1 "AIN2A" H 7623 4121 50  0000 R CNN
 F 2 "connector:Conn_1pin_2.54mm" H 7650 4100 50  0001 C CNN
@@
 $EndComp
 $Comp
-L Connector:Conn_01x01_Male J15
+L Connector:Conn_01x01_Male AIN2B1
 U 1 1 5AE77E1F
 P 7650 4300
-F 0 "J15" H 7350 4300 50  0000 R CNN
+F 0 "AIN2B1" H 7350 4300 50  0000 R CNN
 F 1 "AIN2B" H 7623 4321 50  0000 R CNN
 F 2 "connector:Conn_1pin_2.54mm" H 7650 4300 50  0001 C CNN
@@
 $EndComp
 $Comp
-L Connector:Conn_01x01_Male J16
+L Connector:Conn_01x01_Male AIN3A1
 U 1 1 5AE7846E
 P 7650 4500
-F 0 "J16" H 7350 4500 50  0000 R CNN
+F 0 "AIN3A1" H 7350 4500 50  0000 R CNN
 F 1 "AIN3A" H 7623 4521 50  0000 R CNN
 F 2 "connector:Conn_1pin_2.54mm" H 7650 4500 50  0001 C CNN
@@
 $EndComp
 $Comp
-L Connector:Conn_01x01_Male J17
+L Connector:Conn_01x01_Male AIN3B1
 U 1 1 5AE78ABE
 P 7650 4700
-F 0 "J17" H 7350 4700 50  0000 R CNN
+F 0 "AIN3B1" H 7350 4700 50  0000 R CNN
 F 1 "AIN3B" H 7623 4721 50  0000 R CNN
 F 2 "connector:Conn_1pin_2.54mm" H 7650 4700 50  0001 C CNN
@@
 $EndComp
 $Comp
-L Connector:Conn_01x01_Male J18
+L Connector:Conn_01x01_Male AIN4A1
 U 1 1 5AE7910F
 P 7650 4900
-F 0 "J18" H 7350 4900 50  0000 R CNN
+F 0 "AIN4A1" H 7350 4900 50  0000 R CNN
 F 1 "AIN4A" H 7623 4921 50  0000 R CNN
 F 2 "connector:Conn_1pin_2.54mm" H 7650 4900 50  0001 C CNN
@@
 $EndComp
 $Comp
-L Connector:Conn_01x01_Male J19
+L Connector:Conn_01x01_Male AIN4B1
 U 1 1 5AE79761
 P 7650 5100
-F 0 "J19" H 7350 5100 50  0000 R CNN
+F 0 "AIN4B1" H 7350 5100 50  0000 R CNN
 F 1 "AIN4B" H 7623 5121 50  0000 R CNN
 F 2 "connector:Conn_1pin_2.54mm" H 7650 5100 50  0001 C CNN
@@
 	4550 4450 4950 4450
 $Comp
-L Connector:Conn_01x01_Male J1
+L Connector:Conn_01x01_Male MCLK1
 U 1 1 5AE92C6D
 P 3600 2950
-F 0 "J1" H 3250 2950 50  0000 C CNN
+F 0 "MCLK1" H 3250 2950 50  0000 C CNN
 F 1 "MCLK" H 3500 2950 50  0000 C CNN
 F 2 "connector:Conn_1pin_2.54mm" H 3600 2950 50  0001 C CNN
@@
 $EndComp
 $Comp
-L Connector:Conn_01x01_Male J2
+L Connector:Conn_01x01_Male SCLK1
 U 1 1 5AE92F00
 P 3600 3100
-F 0 "J2" H 3250 3100 50  0000 C CNN
+F 0 "SCLK1" H 3250 3100 50  0000 C CNN
 F 1 "SCLK" H 3500 3100 50  0000 C CNN
 F 2 "connector:Conn_1pin_2.54mm" H 3600 3100 50  0001 C CNN
@@
 $EndComp
 $Comp
-L Connector:Conn_01x01_Male J3
+L Connector:Conn_01x01_Male LRCK1
 U 1 1 5AE94DD9
 P 3600 3250
-F 0 "J3" H 3250 3250 50  0000 C CNN
+F 0 "LRCK1" H 3250 3250 50  0000 C CNN
 F 1 "LRCK" H 3500 3250 50  0000 C CNN
 F 2 "connector:Conn_1pin_2.54mm" H 3600 3250 50  0001 C CNN
@@
 $EndComp
 $Comp
-L Connector:Conn_01x01_Male J4
+L Connector:Conn_01x01_Male SDIN1
 U 1 1 5AE96CB8
 P 3600 3400
-F 0 "J4" H 3250 3400 50  0000 C CNN
+F 0 "SDIN1" H 3250 3400 50  0000 C CNN
 F 1 "SDIN" H 3500 3400 50  0000 C CNN
 F 2 "connector:Conn_1pin_2.54mm" H 3600 3400 50  0001 C CNN
@@
 $EndComp
 $Comp
-L Connector:Conn_01x01_Male J5
+L Connector:Conn_01x01_Male ~RESET1
 U 1 1 5AE98B8F
 P 3600 3550
-F 0 "J5" H 3250 3550 50  0000 C CNN
+F 0 "~RESET1" H 3250 3550 50  0000 C CNN
 F 1 "~RESET" H 3500 3550 50  0000 C CNN
 F 2 "connector:Conn_1pin_2.54mm" H 3600 3550 50  0001 C CNN
@@
 $EndComp
 $Comp
-L Connector:Conn_01x01_Male J6
+L Connector:Conn_01x01_Male SCL1
 U 1 1 5AE9AA74
 P 3600 3700
-F 0 "J6" H 3250 3700 50  0000 C CNN
+F 0 "SCL1" H 3250 3700 50  0000 C CNN
 F 1 "SCL" H 3500 3700 50  0000 C CNN
 F 2 "connector:Conn_1pin_2.54mm" H 3600 3700 50  0001 C CNN
@@
 $EndComp
 $Comp
-L Connector:Conn_01x01_Male J7
+L Connector:Conn_01x01_Male SDA1
 U 1 1 5AE9C957
 P 3600 3850
-F 0 "J7" H 3250 3850 50  0000 C CNN
+F 0 "SDA1" H 3250 3850 50  0000 C CNN
 F 1 "SDA" H 3500 3850 50  0000 C CNN
 F 2 "connector:Conn_1pin_2.54mm" H 3600 3850 50  0001 C CNN

Commit message: Fill out cs43l22 breakout board
Parts:
- added GND1, GND2: GND, connector:Conn_1pin_2.54mm, symbol Connector:Conn_01x01_Male
- added Vcc1: +5V, connector:Conn_1pin_2.54mm, symbol Connector:Conn_01x01_Male
Connections:
- net labels removed: +5V
- wire segments 92 -> 97
Changed lines of the file:
@@
 EESchema Schematic File Version 4
+LIBS:cs43l22_breakout-cache
 EELAYER 26 0
 EELAYER END
@@
 	1450 1350 950  1350
 $Comp
-L power:+5V #PWR020
-U 1 1 5AECA54A
-P 950 1350
-F 0 "#PWR020" H 950 1200 50  0001 C CNN
-F 1 "+5V" V 965 1478 50  0000 L CNN
-F 2 "" H 950 1350 50  0001 C CNN
-F 3 "" H 950 1350 50  0001 C CNN
-	1    950  1350
-	0    -1   -1   0
-$EndComp
-$Comp
 L power:+1V8 #PWR022
 U 1 1 5AECA755
@@
 	1    0    0    -1
 $EndComp
+$Comp
+L Connector:Conn_01x01_Male Vcc1
+U 1 1 5B0B0AAD
+P 750 1350
+F 0 "Vcc1" H 722 1280 50  0000 R CNN
+F 1 "+5V" H 722 1371 50  0000 R CNN
+F 2 "connector:Conn_1pin_2.54mm" H 750 1350 50  0001 C CNN
+F 3 "~" H 750 1350 50  0001 C CNN
+	1    750  1350
+	1    0    0    1
+$EndComp
+$Comp
+L Connector:Conn_01x01_Male GND1
+U 1 1 5B0B0EFF
+P 750 1500
+F 0 "GND1" H 700 1450 50  0000 R CNN
+F 1 "GND" H 722 1521 50  0000 R CNN
+F 2 "connector:Conn_1pin_2.54mm" H 750 1500 50  0001 C CNN
+F 3 "~" H 750 1500 50  0001 C CNN
+	1    750  1500
+	1    0    0    1
+$EndComp
+$Comp
+L Connector:Conn_01x01_Male GND2
+U 1 1 5B0B113B
+P 750 1650
+F 0 "GND2" H 722 1580 50  0000 R CNN
+F 1 "GND" H 722 1671 50  0000 R CNN
+F 2 "connector:Conn_1pin_2.54mm" H 750 1650 50  0001 C CNN
+F 3 "~" H 750 1650 50  0001 C CNN
+	1    750  1650
+	1    0    0    1
+$EndComp
+Wire Wire Line
+	950  1500 1450 1500
+Wire Wire Line
+	1450 1650 1750 1650
+Connection ~ 1750 1650
+Wire Wire Line
+	950  1650 1450 1650
+Connection ~ 1450 1650
+Wire Wire Line
+	1450 1600 1450 1650
+Wire Wire Line
+	1450 1500 1450 1650
 $EndSCHEMATC
