File: hardware/breakout_boards/cs43l22_breakout/cs43l22_breakout.kicad_pcb (KiCad board)
At the start: 2 copper layers, 43 parts, among them J20 SJ-3524, U1 CS43L22_V2, U2 LM1117-1.8

Commit message: Fill out cs43l22 breakout board
Parts:
- removed SDIN1: SDIN, connector:Conn_1pin_2.54mm
- removed SPKR_OUTB+1: SPKR_OUTB+, connector:Conn_1pin_2.54mm
- added GND: GND, connector:Conn_1pin_2.54mm, F.Cu at (83.8, 73.7)
- added GND: GND, connector:Conn_1pin_2.54mm, F.Cu at (109.2, 76.2)
- added SDIN: SDIN, connector:Conn_1pin_2.54mm, F.Cu at (83.8, 81.3)
- added SPKR_OUTB+: SPKR_OUTB+, connector:Conn_1pin_2.54mm, F.Cu at (83.8, 96.5)
- added Vcc: +5V, connector:Conn_1pin_2.54mm, F.Cu at (109.2, 73.7)
- C1, C10, C11, C12, C13, C14, C15, C16, C17, C2, C3, C4, C5, C6, C7, C8, C9, R1, R2, R3, R4: moved to B.Cu
- moved C8 58.1 mm to (103.5, 100.3), turned to 180 degrees
- moved C10 57.7 mm to (103.7, 95.0), turned to 0 degrees
- moved C15 56.4 mm to (103.5, 80.0), turned to 180 degrees
- moved C7 55.3 mm to (103.7, 92.5), turned to 0 degrees
- moved C6 54.4 mm to (103.7, 89.9), turned to 0 degrees
- moved R3 53.8 mm to (95.8, 97.8), turned to 180 degrees
- moved C16 53.3 mm to (103.5, 85.1), turned to 180 degrees
- moved C9 49.3 mm to (103.5, 97.8)
- moved C17 49.3 mm to (103.5, 87.6), turned to 180 degrees
- moved U2 47.2 mm to (96.5, 76.2), turned to 180 degrees
- moved R4 46.2 mm to (95.8, 95.2)
- moved C2 45.6 mm to (95.9, 92.7)
- moved C3 37.6 mm to (88.9, 89.5), turned to 180 degrees
- moved C12 37.2 mm to (88.9, 87.0), turned to 180 degrees
- moved C11 37.1 mm to (88.9, 84.5), turned to 180 degrees
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- renumbered AIN1A1 to AIN1A, AIN1B1 to AIN1B, AIN2A1 to AIN2A, AIN2B1 to AIN2B, AIN3A1 to AIN3A, AIN3B1 to AIN3B, AIN4A1 to AIN4A, AIN4B1 to AIN4B, LRCK1 to LRCK, SCL1 to SCL, SDA1 to SDA, SPKR_OUTA+1 to SPKR_OUTA+, SPKR_OUTA-1 to SPKR_OUTA-, SPKR_OUTB-1 to SPKR_OUTB-, ~RESET1 to ~RESET
Connections:
- U2 pad 3: +5V -> Net-(U2-Pad3)
Routing:
- net GND: track 0.00 -> 72.5 mm, vias 0 -> 8
- net +1V8: track 0.00 -> 71.1 mm, vias 0 -> 8
- net Net-(J20-Pad4): track 0.00 -> 29.7 mm, vias 0 -> 2
- net Net-(C9-Pad2): track 0.00 -> 29.4 mm, vias 0 -> 2
- net Net-(C15-Pad2): track 0.00 -> 28.4 mm, vias 0 -> 1
- net Net-(C8-Pad2): track 0.00 -> 22.7 mm, vias 0 -> 1
- net Net-(R1-Pad1): track 0.00 -> 19.9 mm, vias 0 -> 1
- net Net-(SPKR_OUTB-1-Pad1): track 0.00 -> 16.5 mm
- net Net-(AIN4A1-Pad1): track 0.00 -> 15.8 mm
- net Net-(R2-Pad1): track 0.00 -> 15.4 mm, vias 0 -> 1
- net Net-(SPKR_OUTB+1-Pad1): track 0.00 -> 14.9 mm
- net Net-(MCLK1-Pad1): track 0.00 -> 14.6 mm
- net Net-(AIN4B1-Pad1): track 0.00 -> 13.9 mm
- net Net-(C8-Pad1): track 0.00 -> 13.3 mm
- net Net-(SPKR_OUTA-1-Pad1): track 0.00 -> 13.3 mm
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- added copper zone on F.Cu, net +1V8
- added copper zone on B.Cu, net GND
Other:
- board outline added: 30.5 x 39.4 mm
- net class Default: clearance 0.2 -> 0.1524; trace_width 0.25 -> 0.1524; via_dia 0.8 -> 0.6858; via_drill 0.4 -> 0.3302
- rule trace_clearance: 0.2 -> 0.1524
- rule trace_min: 0.2 -> 0.1524
- rule via_min_drill: 0.3 -> 0.3302
- rule via_min_size: 0.4 -> 0.6858
- board text added: "CS43L22 Breakout Rev. A"

Commit message: Closer cs43l22 edge cuts
Routing:
- net GND: track 72.5 -> 87.5 mm
- net +1V8: track 71.1 -> 83.4 mm, vias 8 -> 9
Other:
- board size 30.5 x 39.4 mm -> 27.9 x 37.3 mm
Changed lines of the file:
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@@
   (general
     (thickness 1.6)
-    (drawings 7)
-    (tracks 313)
+    (drawings 8)
+    (tracks 327)
     (zones 0)
     (modules 46)
@@
       (net 36 "Net-(U2-Pad3)"))
   )
+  (gr_line (start 110.49 109.728) (end 110.49 72.39) (layer Edge.Cuts) (width 0.2))
+  (gr_line (start 110.236 109.728) (end 110.49 109.728) (layer Edge.Cuts) (width 0.2))
+  (gr_line (start 82.55 109.728) (end 110.236 109.728) (layer Edge.Cuts) (width 0.2))
+  (gr_line (start 82.55 72.39) (end 82.55 109.728) (layer Edge.Cuts) (width 0.2))
+  (gr_line (start 82.804 72.39) (end 82.55 72.39) (layer Edge.Cuts) (width 0.2))
+  (gr_line (start 110.49 72.39) (end 82.804 72.39) (layer Edge.Cuts) (width 0.2))
+  (gr_line (start 110.49 73.66) (end 110.49 72.39) (layer Edge.Cuts) (width 0.2))
   (gr_text "CS43L22 Breakout Rev. A" (at 87.884 109.728) (layer F.SilkS)
     (effects (font (size 0.635 0.635) (thickness 0.15875)))
   )
-  (gr_line (start 81.28 110.49) (end 81.28 106.68) (layer Edge.Cuts) (width 0.15))
-  (gr_line (start 111.76 110.49) (end 81.28 110.49) (layer Edge.Cuts) (width 0.15))
-  (gr_line (start 111.76 106.68) (end 111.76 110.49) (layer Edge.Cuts) (width 0.15))
-  (gr_line (start 111.76 71.12) (end 81.28 71.12) (layer Edge.Cuts) (width 0.2))
-  (gr_line (start 111.76 106.68) (end 111.76 71.12) (layer Edge.Cuts) (width 0.2))
-  (gr_line (start 81.28 71.12) (end 81.28 106.68) (layer Edge.Cuts) (width 0.2))
   (segment (start 108.98 73.9) (end 109.22 73.66) (width 0.1524) (layer F.Cu) (net 36))
   (segment (start 99.67 73.9) (end 108.98 73.9) (width 0.1524) (layer F.Cu) (net 36))
@@
   (segment (start 90.17 84.455) (end 90.17 85.2324) (width 0.1524) (layer B.Cu) (net 10))
   (segment (start 91.567 84.455) (end 91.948 84.836) (width 0.1524) (layer B.Cu) (net 10))
-  (via (at 91.948 84.836) (size 0.6858) (drill 0.3302) (layers F.Cu B.Cu) (net 10))
   (segment (start 90.17 84.455) (end 91.567 84.455) (width 0.1524) (layer B.Cu) (net 10))
   (segment (start 93.532928 84.836) (end 93.540428 84.8435) (width 0.1524) (layer F.Cu) (net 10))
-  (segment (start 91.948 84.836) (end 93.532928 84.836) (width 0.1524) (layer F.Cu) (net 10))
   (via (at 94.996 89.408) (size 0.6858) (drill 0.3302) (layers F.Cu B.Cu) (net 11))
   (segment (start 97.155 91.567) (end 94.996 89.408) (width 0.1524) (layer B.Cu) (net 11))
@@
   (segment (start 105.065101 85.420101) (end 104.735 85.09) (width 0.1524) (layer B.Cu) (net 9))
   (segment (start 106.68 85.420101) (end 105.065101 85.420101) (width 0.1524) (layer B.Cu) (net 9))
+  (segment (start 102.806501 75.925679) (end 102.806501 76.898499) (width 0.1524) (layer B.Cu) (net 9))
+  (segment (start 100.322221 73.441399) (end 102.806501 75.925679) (width 0.1524) (layer B.Cu) (net 9))
+  (segment (start 101.942899 77.762101) (end 101.6 78.105) (width 0.1524) (layer B.Cu) (net 9))
+  (segment (start 98.127119 73.441399) (end 100.322221 73.441399) (width 0.1524) (layer B.Cu) (net 9))
+  (segment (start 102.806501 76.898499) (end 101.942899 77.762101) (width 0.1524) (layer B.Cu) (net 9))
+  (segment (start 96.56 75.008518) (end 98.127119 73.441399) (width 0.1524) (layer B.Cu) (net 9))
+  (segment (start 96.56 79.375) (end 96.56 75.008518) (width 0.1524) (layer B.Cu) (net 9))
   (via (at 100.584 91.948) (size 0.6858) (drill 0.3302) (layers F.Cu B.Cu) (net 10))
   (segment (start 101.146 92.51) (end 100.584 91.948) (width 0.1524) (layer B.Cu) (net 10))
@@
   (segment (start 91.948 87.884) (end 91.44 88.392) (width 0.1524) (layer B.Cu) (net 10))
   (segment (start 91.948 84.836) (end 91.948 87.884) (width 0.1524) (layer B.Cu) (net 10))
+  (segment (start 91.948 84.836) (end 93.532928 84.836) (width 0.1524) (layer F.Cu) (net 10))
+  (via (at 91.948 84.836) (size 0.6858) (drill 0.3302) (layers F.Cu B.Cu) (net 10) (status 1000000))
+  (segment (start 93.599 84.836) (end 91.948 84.836) (width 0.1524) (layer B.Cu) (net 10))
+  (segment (start 97.79 80.645) (end 93.599 84.836) (width 0.1524) (layer B.Cu) (net 10))
+  (via (at 97.282 93.98) (size 0.6858) (drill 0.3302) (layers F.Cu B.Cu) (net 10))
+  (segment (start 96.176399 93.517881) (end 96.638518 93.98) (width 0.1524) (layer B.Cu) (net 10))
+  (segment (start 96.176399 91.437011) (end 96.176399 93.517881) (width 0.1524) (layer B.Cu) (net 10))
+  (segment (start 95.2265 90.487112) (end 96.176399 91.437011) (width 0.1524) (layer B.Cu) (net 10))
+  (segment (start 96.638518 93.98) (end 97.282 93.98) (width 0.1524) (layer B.Cu) (net 10))
   (via (at 93.141797 89.408) (size 0.6858) (drill 0.3302) (layers F.Cu B.Cu) (net 13))
   (segment (start 93.141797 89.400381) (end 93.141797 89.408) (width 0.1524) (layer F.Cu) (net 13))
@@
   (segment (start 92.011501 87.970027) (end 92.011501 90.868499) (width 0.1524) (layer F.Cu) (net 32))
   (segment (start 92.011501 90.868499) (end 84.619999 98.260001) (width 0.1524) (layer F.Cu) (net 32))
-  (zone (net 10) (net_name +1V8) (layer F.Cu) (hatch edge 0.508)
-    (connect_pads (clearance 0.508))
-    (min_thickness 0.254)
-    (fill yes (arc_segments 16) (thermal_gap 0.508) (thermal_bridge_width 0.508))
-    (polygon
-      (pts
-        (xy 81.915 71.755) (xy 81.915 109.855) (xy 111.125 109.855) (xy 111.125 71.755)
-      )
-    )
-  )
   (zone (net 9) (net_name GND) (layer B.Cu) (hatch edge 0.508)
     (connect_pads (clearance 0.508))
@@
       )
     )
+  )
+  (zone (net 10) (net_name +1V8) (layer F.Cu) (hatch edge 0.508)
+    (connect_pads (clearance 0.508))
+    (min_thickness 0.254)
+    (fill yes (arc_segments 16) (thermal_gap 0.508) (thermal_bridge_width 0.508))
+    (polygon
+      (pts
+        (xy 110.236 72.644) (xy 82.55 72.39) (xy 82.55 109.728) (xy 110.236 109.474)
+      )
+    )
