File: clock/hardware/clock/clock.kicad_pcb (KiCad board)
At the start: 2 copper layers, 45.7 x 58.4 mm, 27 parts, among them J1 USB_B_Micro, J2 7SEG_DEBUG, J3 Conn_ARM_JTAG_SWD_10, U1 LM1117-3.3, U2 AS1115, U3 LTC-4727JS, U4 STM32L151C8TxA, Y1 32.768kHz

Commit message: Minor track cleanup.
Routing:
- net +3V3: track 208.8 -> 201.0 mm, vias 11 -> 10
- net GND: track 96.1 -> 95.9 mm, vias 9 -> 12
Other:
- net class GndRail: trace_width 0.4 -> 0.1524
Changed lines of the file:
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@@
     (thickness 1.6)
     (drawings 9)
-    (tracks 329)
+    (tracks 343)
     (zones 0)
     (modules 27)
@@
   (net_class GndRail ""
     (clearance 0.1524)
-    (trace_width 0.4)
+    (trace_width 0.1524)
     (via_dia 0.6858)
     (via_drill 0.3302)
@@
   (segment (start 84.1375 29.877182) (end 84.76973 30.509412) (width 0.1524) (layer B.Cu) (net 1))
   (segment (start 84.1375 29.0957) (end 84.1375 29.877182) (width 0.1524) (layer B.Cu) (net 1))
-  (via (at 90.17 21.59) (size 0.6858) (drill 0.3302) (layers F.Cu B.Cu) (net 1))
   (segment (start 87.63 21.59) (end 90.17 21.59) (width 0.1524) (layer B.Cu) (net 1))
   (via (at 71.12 27.94) (size 0.6858) (drill 0.3302) (layers F.Cu B.Cu) (net 1))
@@
   (segment (start 99.22 37.94) (end 99.06 38.1) (width 0.1524) (layer B.Cu) (net 1))
   (segment (start 99.22 36.83) (end 99.22 37.94) (width 0.1524) (layer B.Cu) (net 1))
-  (via (at 69.85 39.37) (size 0.6858) (drill 0.3302) (layers F.Cu B.Cu) (net 1))
-  (segment (start 71.14 40.66) (end 69.85 39.37) (width 0.1524) (layer B.Cu) (net 1))
-  (segment (start 71.14 41.91) (end 71.14 40.66) (width 0.1524) (layer B.Cu) (net 1))
   (segment (start 79.47 49.74) (end 78.6676 49.74) (width 0.1524) (layer F.Cu) (net 1))
   (via (at 78.74 43.18) (size 0.6858) (drill 0.3302) (layers F.Cu B.Cu) (net 1))
@@
   (segment (start 91.44 52.07) (end 90.17 53.34) (width 0.1524) (layer B.Cu) (net 1))
   (segment (start 90.17 53.34) (end 85.09 53.34) (width 0.1524) (layer B.Cu) (net 1))
-  (segment (start 96.272401 44.788079) (end 95.239021 43.754699) (width 0.4) (layer F.Cu) (net 1))
-  (segment (start 97.79 61.57) (end 97.79 61.32) (width 0.4) (layer F.Cu) (net 1))
-  (segment (start 95.537599 53.439802) (end 96.272401 52.705) (width 0.4) (layer F.Cu) (net 1))
-  (segment (start 97.79 60.17) (end 95.537599 57.917599) (width 0.4) (layer F.Cu) (net 1))
-  (segment (start 97.79 61.57) (end 97.79 60.17) (width 0.4) (layer F.Cu) (net 1))
-  (segment (start 96.272401 52.705) (end 96.272401 44.788079) (width 0.4) (layer F.Cu) (net 1))
-  (segment (start 95.537599 57.917599) (end 95.537599 53.439802) (width 0.4) (layer F.Cu) (net 1))
-  (segment (start 96.272401 27.692401) (end 90.17 21.59) (width 0.4) (layer F.Cu) (net 1))
   (segment (start 74.355301 24.704699) (end 71.462899 27.597101) (width 0.4) (layer F.Cu) (net 1))
   (segment (start 71.462899 27.597101) (end 71.12 27.94) (width 0.4) (layer F.Cu) (net 1))
-  (segment (start 87.63 21.59) (end 84.515301 24.704699) (width 0.4) (layer F.Cu) (net 1))
   (segment (start 69.85 29.21) (end 71.12 27.94) (width 0.4) (layer F.Cu) (net 1))
-  (segment (start 67.31 41.91) (end 65.95 41.91) (width 0.4) (layer F.Cu) (net 1))
-  (segment (start 69.85 39.37) (end 67.31 41.91) (width 0.4) (layer F.Cu) (net 1))
   (via (at 83.637203 27.487797) (size 0.6858) (drill 0.3302) (layers F.Cu B.Cu) (net 1))
   (segment (start 97.155 40.005) (end 99.06 38.1) (width 0.4) (layer F.Cu) (net 1))
   (segment (start 96.272401 40.005) (end 97.155 40.005) (width 0.4) (layer F.Cu) (net 1))
-  (segment (start 96.272401 52.705) (end 96.272401 40.005) (width 0.4) (layer F.Cu) (net 1))
   (segment (start 96.272401 40.005) (end 96.272401 27.692401) (width 0.4) (layer F.Cu) (net 1))
   (segment (start 85.07 51.34) (end 85.07 53.32) (width 0.1524) (layer F.Cu) (net 1))
@@
   (segment (start 78.74 43.18) (end 73.1474 43.18) (width 0.1524) (layer B.Cu) (net 1))
   (segment (start 69.85 29.21) (end 62.23 36.83) (width 0.4) (layer F.Cu) (net 1))
-  (segment (start 62.23 36.83) (end 62.23 52.07) (width 0.4) (layer F.Cu) (net 1))
   (via (at 78.74 53.975) (size 0.6858) (drill 0.3302) (layers F.Cu B.Cu) (net 1))
   (segment (start 64.135 53.975) (end 78.74 53.975) (width 0.4) (layer F.Cu) (net 1))
@@
   (segment (start 83.185 24.704699) (end 74.355301 24.704699) (width 0.4) (layer F.Cu) (net 1))
   (segment (start 84.515301 24.704699) (end 83.185 24.704699) (width 0.4) (layer F.Cu) (net 1))
+  (segment (start 95.19 43.18) (end 95.09 43.18) (width 0.4) (layer F.Cu) (net 1))
+  (segment (start 96.272401 44.262401) (end 95.19 43.18) (width 0.4) (layer F.Cu) (net 1))
+  (segment (start 97.79 61.57) (end 97.79 61.32) (width 0.4) (layer F.Cu) (net 1))
+  (segment (start 93.98 54.997401) (end 96.272401 52.705) (width 0.4) (layer F.Cu) (net 1))
+  (segment (start 97.79 61.32) (end 93.98 57.51) (width 0.4) (layer F.Cu) (net 1))
+  (segment (start 96.272401 52.705) (end 96.272401 44.262401) (width 0.4) (layer F.Cu) (net 1))
+  (segment (start 93.98 57.51) (end 93.98 54.997401) (width 0.4) (layer F.Cu) (net 1))
+  (segment (start 96.272401 40.947599) (end 96.272401 40.005) (width 0.4) (layer F.Cu) (net 1))
+  (segment (start 95.09 42.13) (end 96.272401 40.947599) (width 0.4) (layer F.Cu) (net 1))
+  (segment (start 95.09 43.18) (end 95.09 42.13) (width 0.4) (layer F.Cu) (net 1))
+  (segment (start 96.272401 27.692401) (end 91.44 22.86) (width 0.4) (layer F.Cu) (net 1))
+  (segment (start 86.36 22.86) (end 84.515301 24.704699) (width 0.4) (layer F.Cu) (net 1))
+  (via (at 90.17 21.59) (size 0.6858) (drill 0.3302) (layers F.Cu B.Cu) (net 1))
+  (segment (start 90.17 22.86) (end 90.17 21.59) (width 0.4) (layer F.Cu) (net 1))
+  (segment (start 91.44 22.86) (end 90.17 22.86) (width 0.4) (layer F.Cu) (net 1))
+  (segment (start 90.17 22.86) (end 86.36 22.86) (width 0.4) (layer F.Cu) (net 1))
+  (segment (start 64.5674 40.005) (end 62.23 40.005) (width 0.1524) (layer F.Cu) (net 1))
+  (segment (start 65.95 41.3876) (end 64.5674 40.005) (width 0.1524) (layer F.Cu) (net 1))
+  (segment (start 65.95 41.91) (end 65.95 41.3876) (width 0.1524) (layer F.Cu) (net 1))
+  (segment (start 62.23 36.83) (end 62.23 40.005) (width 0.4) (layer F.Cu) (net 1))
+  (segment (start 62.23 40.005) (end 62.23 52.07) (width 0.4) (layer F.Cu) (net 1))
   (segment (start 76.174589 36.228255) (end 76.17459 37.431746) (width 0.1524) (layer B.Cu) (net 2))
   (segment (start 84.1375 34.4043) (end 84.1375 33.4519) (width 0.1524) (layer B.Cu) (net 2))
@@
   (segment (start 65.95 43.18) (end 65.95 44.45) (width 0.1524) (layer F.Cu) (net 2))
   (segment (start 76.78 63.5) (end 76.82 63.46) (width 0.1524) (layer F.Cu) (net 2))
-  (segment (start 71.12 63.5) (end 76.78 63.5) (width 0.1524) (layer F.Cu) (net 2))
   (segment (start 95.49 61.82) (end 95.49 61.57) (width 0.4) (layer F.Cu) (net 2))
   (segment (start 95.49 61.57) (end 95.49 62.47) (width 0.4) (layer F.Cu) (net 2))
@@
   (segment (start 92.075 67.31) (end 95.25 64.135) (width 0.4) (layer B.Cu) (net 2))
   (segment (start 92.075 67.945) (end 92.075 67.31) (width 0.4) (layer B.Cu) (net 2))
+  (via (at 70.485 65.405) (size 0.6858) (drill 0.3302) (layers F.Cu B.Cu) (net 2))
+  (segment (start 71.12 64.77) (end 70.485 65.405) (width 0.1524) (layer F.Cu) (net 2))
+  (segment (start 71.12 63.5) (end 71.12 64.77) (width 0.1524) (layer F.Cu) (net 2))
+  (via (at 71.755 58.42) (size 0.6858) (drill 0.3302) (layers F.Cu B.Cu) (net 2))
+  (segment (start 71.6126 58.42) (end 71.755 58.42) (width 0.1524) (layer F.Cu) (net 2))
+  (segment (start 71.12 58.9126) (end 71.6126 58.42) (width 0.1524) (layer F.Cu) (net 2))
+  (segment (start 71.12 59.69) (end 71.12 58.9126) (width 0.1524) (layer F.Cu) (net 2))
+  (via (at 103.505 49.53) (size 0.6858) (drill 0.3302) (layers F.Cu B.Cu) (net 2))
+  (segment (start 103.7524 49.53) (end 103.505 49.53) (width 0.1524) (layer F.Cu) (net 2))
+  (segment (start 104.22 49.0624) (end 103.7524 49.53) (width 0.1524) (layer F.Cu) (net 2))
+  (segment (start 104.22 48.26) (end 104.22 49.0624) (width 0.1524) (layer F.Cu) (net 2))
   (segment (start 69.398601 54.701399) (end 68.62 55.48) (width 0.1524) (layer F.Cu) (net 3))
   (segment (start 79.395083 54.701399) (end 69.398601 54.701399) (width 0.1524) (layer F.Cu) (net 3))
@@
   (segment (start 78.8324 55.88) (end 82.57 52.1424) (width 0.1524) (layer F.Cu) (net 4))
   (segment (start 71.12 55.88) (end 78.8324 55.88) (width 0.1524) (layer F.Cu) (net 4))
+  (segment (start 71.12 55.88) (end 71.12 56.9824) (width 0.1524) (layer F.Cu) (net 4))
+  (segment (start 71.12 56.9824) (end 69.85 58.2524) (width 0.1524) (layer F.Cu) (net 4))
+  (segment (start 69.85 61.4926) (end 68.62 62.7226) (width 0.1524) (layer F.Cu) (net 4))
   (segment (start 68.62 62.7226) (end 68.62 63.5) (width 0.1524) (layer F.Cu) (net 4))
-  (segment (start 69.598601 61.743999) (end 68.62 62.7226) (width 0.1524) (layer F.Cu) (net 4))
-  (segment (start 69.598601 58.503799) (end 69.598601 61.743999) (width 0.1524) (layer F.Cu) (net 4))
-  (segment (start 71.12 56.9824) (end 69.598601 58.503799) (width 0.1524) (layer F.Cu) (net 4))
-  (segment (start 71.12 55.88) (end 71.12 56.9824) (width 0.1524) (layer F.Cu) (net 4))
+  (segment (start 69.85 58.2524) (end 69.85 61.4926) (width 0.1524) (layer F.Cu) (net 4))
   (segment (start 97.79 43.18) (end 101.44 43.18) (width 0.1524) (layer F.Cu) (net 5))
   (segment (start 97.87 48.26) (end 101.52 48.26) (width 0.1524) (layer F.Cu) (net 6))
