File: clock/hardware/clock/clock.sch (KiCad schematic (older format))
At the start: 23 parts

Commit message: More clock schematic work
Parts:
- removed D?: LED Blue, LED_THT:LED_D3.0mm_IRBlack, symbol LED:TSAL4400
- removed D?: LED Green, LED_THT:LED_D3.0mm_IRBlack, symbol LED:TSAL4400
- removed D?: LED Red, LED_THT:LED_D3.0mm_IRBlack, symbol LED:TSAL4400
- added C8: 0.1uf, symbol pspice:C
- added D1: LED Blue, symbol Device:LED
- added D2: LED Green, symbol Device:LED
- added D3: LED Red, symbol Device:LED
- added J3: Conn_ARM_JTAG_SWD_10, Connector_PinHeader_1.27mm:PinHeader_2x05_P1.27mm_Vertical_SMD, symbol Connector:Conn_ARM_JTAG_SWD_10
- added R4: 10k, symbol pspice:R
- added Y1: 32.768kHz, symbol Device:Crystal
- gave numbers to parts that had none: 20
Connections:
- net labels added: JTAG_RST, JTAG_TCK, JTAG_TDI, JTAG_TDO, JTAG_TMS
- wire segments 133 -> 157
Other:
- moved on the sheet: C7

Commit message: Assign clock footprints
Parts:
- removed C8: 0.1uf, symbol pspice:C
- C1, C2, C6, C7: footprint (none) -> Capacitors_SMD:C_0805_HandSoldering
- C3: renamed from C4; footprint (none) -> Capacitors_SMD:C_0805_HandSoldering
- C4: renamed from C5; footprint (none) -> Capacitors_SMD:C_0805_HandSoldering
- D1, D2, D3: footprint (none) -> LEDs:LED_0805_HandSoldering
- J1: footprint (none) -> Connectors:USB_Micro-B_10103594-0001LF
- R4: footprint (none) -> Resistors_SMD:R_0805_HandSoldering
- R5, R6, R7: value 60 -> 300; footprint (none) -> Resistors_SMD:R_0805_HandSoldering
- S1: footprint (none) -> nome:PEC11
- U1: footprint (none) -> TO_SOT_Packages_SMD:SOT-223
- Y1: footprint (none) -> crystal:ECS-31B_xtal
- renumbered C3 to C5
Connections:
- net labels removed: +5V, JTAG_RST, JTAG_TDI, JTAG_TDO
- wire segments 157 -> 147
- no-connect marks 12 -> 15
Changed lines of the file:
@@
 EESchema Schematic File Version 4
-LIBS:as1115_display_breakout-cache
+LIBS:clock-cache
 EELAYER 26 0
 EELAYER END
@@
 $EndComp
 $Comp
-L pspice:C C3
+L pspice:C C5
 U 1 1 59EC7FF1
 P 2100 2200
-F 0 "C3" H 2125 2300 50  0000 L CNN
+F 0 "C5" H 2125 2300 50  0000 L CNN
 F 1 "0.1uF" H 2125 2100 50  0000 L CNN
 F 2 "Capacitors_SMD:C_0805_HandSoldering" H 2138 2050 50  0001 C CNN
@@
 7SEG_SCL
 $Comp
-L power:+5V #PWR04
+L power:+3V3 #PWR04
 U 1 1 5AE16CF3
 P 2100 1200
 F 0 "#PWR04" H 2100 1050 50  0001 C CNN
-F 1 "+5V" H 2115 1373 50  0000 C CNN
+F 1 "+3V3" H 2115 1373 50  0000 C CNN
 F 2 "" H 2100 1200 50  0001 C CNN
 F 3 "" H 2100 1200 50  0001 C CNN
@@
 $EndComp
 $Comp
-L power:+5V #PWR07
+L power:+3V3 #PWR07
 U 1 1 5AE17CF5
 P 2750 800
 F 0 "#PWR07" H 2750 650 50  0001 C CNN
-F 1 "+5V" H 2765 973 50  0000 C CNN
+F 1 "+3V3" H 2765 973 50  0000 C CNN
 F 2 "" H 2750 800 50  0001 C CNN
 F 3 "" H 2750 800 50  0001 C CNN
@@
 Connection ~ 2750 800
 $Comp
-L power:+5V #PWR08
+L power:+3V3 #PWR08
 U 1 1 5AE17D2F
 P 2950 800
 F 0 "#PWR08" H 2950 650 50  0001 C CNN
-F 1 "+5V" H 2965 973 50  0000 C CNN
+F 1 "+3V3" H 2965 973 50  0000 C CNN
 F 2 "" H 2950 800 50  0001 C CNN
 F 3 "" H 2950 800 50  0001 C CNN
@@
 P 11300 2400
 F 0 "R5" H 11368 2446 50  0000 L CNN
-F 1 "60" H 11368 2355 50  0000 L CNN
-F 2 "" H 11300 2400 50  0001 C CNN
+F 1 "300" H 11368 2355 50  0000 L CNN
+F 2 "Resistors_SMD:R_0805_HandSoldering" H 11300 2400 50  0001 C CNN
 F 3 "" H 11300 2400 50  0001 C CNN
 	1    11300 2400
@@
 P 11950 2400
 F 0 "R6" H 12018 2446 50  0000 L CNN
-F 1 "60" H 12018 2355 50  0000 L CNN
-F 2 "" H 11950 2400 50  0001 C CNN
+F 1 "300" H 12018 2355 50  0000 L CNN
+F 2 "Resistors_SMD:R_0805_HandSoldering" H 11950 2400 50  0001 C CNN
 F 3 "" H 11950 2400 50  0001 C CNN
 	1    11950 2400
@@
 P 12600 2400
 F 0 "R7" H 12668 2446 50  0000 L CNN
-F 1 "60" H 12668 2355 50  0000 L CNN
-F 2 "" H 12600 2400 50  0001 C CNN
+F 1 "300" H 12668 2355 50  0000 L CNN
+F 2 "Resistors_SMD:R_0805_HandSoldering" H 12600 2400 50  0001 C CNN
 F 3 "" H 12600 2400 50  0001 C CNN
 	1    12600 2400
@@
 F 0 "C1" H 1528 5046 50  0000 L CNN
 F 1 "0.1uf" H 1528 4955 50  0000 L CNN
-F 2 "" H 1350 5000 50  0001 C CNN
+F 2 "Capacitors_SMD:C_0805_HandSoldering" H 1350 5000 50  0001 C CNN
 F 3 "" H 1350 5000 50  0001 C CNN
 	1    1350 5000
@@
 F 0 "C2" H 2028 5046 50  0000 L CNN
 F 1 "0.1uf" H 2028 4955 50  0000 L CNN
-F 2 "" H 1850 5000 50  0001 C CNN
+F 2 "Capacitors_SMD:C_0805_HandSoldering" H 1850 5000 50  0001 C CNN
 F 3 "" H 1850 5000 50  0001 C CNN
 	1    1850 5000
@@
 $EndComp
 $Comp
-L pspice:C C4
+L pspice:C C3
 U 1 1 5AE70AD7
 P 2400 5000
-F 0 "C4" H 2578 5046 50  0000 L CNN
+F 0 "C3" H 2578 5046 50  0000 L CNN
 F 1 "0.1uf" H 2578 4955 50  0000 L CNN
-F 2 "" H 2400 5000 50  0001 C CNN
+F 2 "Capacitors_SMD:C_0805_HandSoldering" H 2400 5000 50  0001 C CNN
 F 3 "" H 2400 5000 50  0001 C CNN
 	1    2400 5000
@@
 $EndComp
 $Comp
-L pspice:C C5
+L pspice:C C4
 U 1 1 5AE70B32
 P 2900 5000
-F 0 "C5" H 3078 5046 50  0000 L CNN
+F 0 "C4" H 3078 5046 50  0000 L CNN
 F 1 "0.1uf" H 3078 4955 50  0000 L CNN
-F 2 "" H 2900 5000 50  0001 C CNN
+F 2 "Capacitors_SMD:C_0805_HandSoldering" H 2900 5000 50  0001 C CNN
 F 3 "" H 2900 5000 50  0001 C CNN
 	1    2900 5000
@@
 F 0 "J1" H 1055 7617 50  0000 C CNN
 F 1 "USB_B_Micro" H 1055 7526 50  0000 C CNN
-F 2 "" H 1150 7100 50  0001 C CNN
+F 2 "Connectors:USB_Micro-B_10103594-0001LF" H 1150 7100 50  0001 C CNN
 F 3 "~" H 1150 7100 50  0001 C CNN
 	1    1000 7150
@@
 	1    0    0    -1
 $EndComp
-Wire Wire Line
-	1300 6950 1700 6950
-Wire Wire Line
-	1700 6950 1700 6800
-$Comp
-L power:+5V #PWR03
-U 1 1 5AE97FFC
-P 1700 6800
-F 0 "#PWR03" H 1700 6650 50  0001 C CNN
-F 1 "+5V" H 1715 6973 50  0000 C CNN
-F 2 "" H 1700 6800 50  0001 C CNN
-F 3 "" H 1700 6800 50  0001 C CNN
-	1    1700 6800
-	1    0    0    -1
-$EndComp
 NoConn ~ 1300 7150
 NoConn ~ 1300 7250
@@
 F 0 "U1" H 2300 7192 50  0000 C CNN
 F 1 "LM1117-3.3" H 2300 7101 50  0000 C CNN
-F 2 "" H 2300 6950 50  0001 C CNN
+F 2 "TO_SOT_Packages_SMD:SOT-223" H 2300 6950 50  0001 C CNN
 F 3 "http://www.ti.com/lit/ds/symlink/lm1117.pdf" H 2300 6950 50  0001 C CNN
 	1    2300 6950
 	1    0    0    -1
 $EndComp
-Wire Wire Line
-	1700 6950 2000 6950
-Connection ~ 1700 6950
 Wire Wire Line
 	2300 7250 2300 7450
@@
 F 0 "S1" H 14378 7203 60  0000 L CNN
 F 1 "PEC11R" H 14378 7097 60  0000 L CNN
-F 2 "" H 14150 7150 60  0001 C CNN
+F 2 "nome:PEC11" H 14150 7150 60  0001 C CNN
 F 3 "" H 14150 7150 60  0001 C CNN
 	1    14150 7150
@@
 F 0 "C6" V 3585 6150 50  0000 C CNN
 F 1 "10pf" V 3676 6150 50  0000 C CNN
-F 2 "" H 3900 6150 50  0001 C CNN
+F 2 "Capacitors_SMD:C_0805_HandSoldering" H 3900 6150 50  0001 C CNN
 F 3 "" H 3900 6150 50  0001 C CNN
 	1    3900 6150
@@
 F 0 "C7" V 3585 6650 50  0000 C CNN
 F 1 "10pf" V 3676 6650 50  0000 C CNN
-F 2 "" H 3900 6650 50  0001 C CNN
+F 2 "Capacitors_SMD:C_0805_HandSoldering" H 3900 6650 50  0001 C CNN
 F 3 "" H 3900 6650 50  0001 C CNN
 	1    3900 6650
@@
 F 0 "Y1" V 4100 6550 50  0000 L CNN
 F 1 "32.768kHz" V 4200 6550 50  0000 L CNN
-F 2 "" H 4200 6400 50  0001 C CNN
+F 2 "crystal:ECS-31B_xtal" H 4200 6400 50  0001 C CNN
 F 3 "~" H 4200 6400 50  0001 C CNN
 	1    4200 6400
@@
 F 0 "D1" V 11338 1783 50  0000 R CNN
 F 1 "LED Blue" V 11247 1783 50  0000 R CNN
-F 2 "" H 11300 1900 50  0001 C CNN
+F 2 "LEDs:LED_0805_HandSoldering" H 11300 1900 50  0001 C CNN
 F 3 "~" H 11300 1900 50  0001 C CNN
 	1    11300 1900
@@
 F 0 "D2" V 11988 1783 50  0000 R CNN
 F 1 "LED Green" V 11897 1783 50  0000 R CNN
-F 2 "" H 11950 1900 50  0001 C CNN
+F 2 "LEDs:LED_0805_HandSoldering" H 11950 1900 50  0001 C CNN
 F 3 "~" H 11950 1900 50  0001 C CNN
 	1    11950 1900
@@
 F 0 "D3" V 12638 1783 50  0000 R CNN
 F 1 "LED Red" V 12547 1783 50  0000 R CNN
-F 2 "" H 12600 1900 50  0001 C CNN
+F 2 "LEDs:LED_0805_HandSoldering" H 12600 1900 50  0001 C CNN
 F 3 "~" H 12600 1900 50  0001 C CNN
 	1    12600 1900
@@
 	1    0    0    -1
 $EndComp
-$Comp
-L pspice:C C8
-U 1 1 5AF34021
-P 4200 5700
-F 0 "C8" H 4378 5746 50  0000 L CNN
-F 1 "0.1uf" H 4378 5655 50  0000 L CNN
-F 2 "" H 4200 5700 50  0001 C CNN
-F 3 "" H 4200 5700 50  0001 C CNN
-	1    4200 5700
-	1    0    0    -1
-$EndComp
-$Comp
-L power:GND #PWR012
-U 1 1 5AF34107
-P 4200 5950
-F 0 "#PWR012" H 4200 5700 50  0001 C CNN
-F 1 "GND" H 4205 5777 50  0000 C CNN
-F 2 "" H 4200 5950 50  0001 C CNN
-F 3 "" H 4200 5950 50  0001 C CNN
-	1    4200 5950
-	1    0    0    -1
-$EndComp
-Text Label 3950 5350 0    50   ~ 0
-JTAG_RST
-Wire Wire Line
-	15200 3950 15450 3950
-Text Label 15450 3950 0    50   ~ 0
-JTAG_RST
-Wire Wire Line
-	3950 5350 4200 5350
-Wire Wire Line
-	4200 5450 4200 5350
-Connection ~ 4200 5350
-Wire Wire Line
-	4200 5350 5100 5350
 Wire Wire Line
 	15200 4250 15450 4250
@@
 Text Label 15450 4150 0    50   ~ 0
 JTAG_TCK
-Wire Wire Line
-	15200 4350 15450 4350
-Text Label 15450 4350 0    50   ~ 0
-JTAG_TDO
-Wire Wire Line
-	15200 4450 15450 4450
-Text Label 15450 4450 0    50   ~ 0
-JTAG_TDI
 Wire Wire Line
 	14700 3650 14700 3400
@@
 Text Label 12600 8050 0    50   ~ 0
 JTAG_TCK
-Wire Wire Line
-	12300 8150 12600 8150
-Text Label 12600 8150 0    50   ~ 0
-JTAG_TDI
-Wire Wire Line
-	5100 6950 4600 6950
-Text Label 4600 6950 0    50   ~ 0
-JTAG_TDO
 $Comp
 L pspice:R R4
@@
 F 0 "R4" H 4818 5896 50  0000 L CNN
 F 1 "10k" H 4818 5805 50  0000 L CNN
-F 2 "" H 4750 5850 50  0001 C CNN
+F 2 "Resistors_SMD:R_0805_HandSoldering" H 4750 5850 50  0001 C CNN
 F 3 "" H 4750 5850 50  0001 C CNN
 	1    4750 5850
@@
 Wire Wire Line
 	4750 5550 4750 5600
+Wire Wire Line
+	1300 6950 2000 6950
+NoConn ~ 15200 4350
+NoConn ~ 15200 4450
+NoConn ~ 15200 3950
 $EndSCHEMATC

Commit message: Start laying out clock footprints
Parts:
- J3: footprint Connector_PinHeader_1.27mm:PinHeader_2x05_P1.27mm_Vertical_SMD -> Pin_Headers:Pin_Header_Straight_2x05_Pitch1.27mm
- U4: footprint Package_QFP:LQFP-48_7x7mm_P0.5mm -> Housings_QFP:LQFP-48_7x7mm_Pitch0.5mm
Changed lines of the file:
@@
 F 0 "U4" H 8700 8728 50  0000 C CNN
 F 1 "STM32L151C8TxA" H 8700 8637 50  0000 C CNN
-F 2 "Package_QFP:LQFP-48_7x7mm_P0.5mm" H 12200 8425 50  0001 R TNN
+F 2 "Housings_QFP:LQFP-48_7x7mm_Pitch0.5mm" H 12200 8425 50  0001 R TNN
 F 3 "http://www.st.com/st-web-ui/static/active/en/resource/technical/document/datasheet/CD00277537.pdf" H 8700 6750 50  0001 C CNN
 	1    8700 6750
@@
 Wire Wire Line
 	3000 1400 3850 1400
-Wire Wire Line
-	3500 1500 3650 1500
 $Comp
 L power:GND #PWR016
@@
 F 0 "J3" H 14260 4296 50  0000 R CNN
 F 1 "Conn_ARM_JTAG_SWD_10" H 14260 4205 50  0000 R CNN
-F 2 "Connector_PinHeader_1.27mm:PinHeader_2x05_P1.27mm_Vertical_SMD" H 14750 3700 50  0001 L TNN
+F 2 "Pin_Headers:Pin_Header_Straight_2x05_Pitch1.27mm" H 14750 3700 50  0001 L TNN
 F 3 "http://infocenter.arm.com/help/topic/com.arm.doc.faqs/attached/13634/cortex_debug_connectors.pdf" V 14350 3000 50  0001 C CNN
 	1    14700 4250
@@
 NoConn ~ 15200 4450
 NoConn ~ 15200 3950
+Wire Wire Line
+	3500 1500 3850 1500
 $EndSCHEMATC

Commit message: Change to non-slotted USB connector
Parts:
- J1: footprint Connectors:USB_Micro-B_10103594-0001LF -> custom_connectors:10118192-0001LF
Changed lines of the file:
@@
 F 0 "J1" H 1055 7617 50  0000 C CNN
 F 1 "USB_B_Micro" H 1055 7526 50  0000 C CNN
-F 2 "Connectors:USB_Micro-B_10103594-0001LF" H 1150 7100 50  0001 C CNN
+F 2 "custom_connectors:10118192-0001LF" H 1150 7100 50  0001 C CNN
 F 3 "~" H 1150 7100 50  0001 C CNN
 	1    1000 7150

Commit message: Rev B. of clock. Power rails. SMD JTAG connector.
Parts:
- J3: footprint Pin_Headers:Pin_Header_Straight_2x05_Pitch1.27mm -> Pin_Headers:Pin_Header_Straight_2x05_Pitch1.27mm_SMD
- U4: symbol MCU_ST_STM32:STM32L151C8TxA -> clock-rescue:STM32L151C8TxA-MCU_ST_STM32
Connections:
- wire segments 147 -> 140
- no-connect marks 15 -> 17
Changed lines of the file:
@@
 	2950 1800 3850 1800
 $Comp
-L MCU_ST_STM32:STM32L151C8TxA U4
+L clock-rescue:STM32L151C8TxA-MCU_ST_STM32 U4
 U 1 1 5AE146A0
 P 8700 6750
@@
 	1    0    0    -1
 $EndComp
-Wire Wire Line
-	1000 7550 1000 7650
 $Comp
 L power:GND #PWR01
@@
 NoConn ~ 1300 7150
 NoConn ~ 1300 7250
-Wire Wire Line
-	900  7550 900  7650
-Wire Wire Line
-	900  7650 1000 7650
-Connection ~ 1000 7650
-Wire Wire Line
-	1000 7650 1000 7800
 NoConn ~ 1300 7350
 $Comp
@@
 F 0 "J3" H 14260 4296 50  0000 R CNN
 F 1 "Conn_ARM_JTAG_SWD_10" H 14260 4205 50  0000 R CNN
-F 2 "Pin_Headers:Pin_Header_Straight_2x05_Pitch1.27mm" H 14750 3700 50  0001 L TNN
+F 2 "Pin_Headers:Pin_Header_Straight_2x05_Pitch1.27mm_SMD" H 14750 3700 50  0001 L TNN
 F 3 "http://infocenter.arm.com/help/topic/com.arm.doc.faqs/attached/13634/cortex_debug_connectors.pdf" V 14350 3000 50  0001 C CNN
 	1    14700 4250
@@
 $EndComp
 Wire Wire Line
-	14600 4850 14600 5050
-Wire Wire Line
-	14600 5050 14650 5050
-Wire Wire Line
 	14700 5050 14700 4850
-Wire Wire Line
-	14650 5050 14650 5200
-Connection ~ 14650 5050
-Wire Wire Line
-	14650 5050 14700 5050
 $Comp
 L power:GND #PWR020
 U 1 1 5AF2E1E1
-P 14650 5200
-F 0 "#PWR020" H 14650 4950 50  0001 C CNN
-F 1 "GND" H 14655 5027 50  0000 C CNN
-F 2 "" H 14650 5200 50  0001 C CNN
-F 3 "" H 14650 5200 50  0001 C CNN
-	1    14650 5200
+P 14700 5050
+F 0 "#PWR020" H 14700 4800 50  0001 C CNN
+F 1 "GND" H 14705 4877 50  0000 C CNN
+F 2 "" H 14700 5050 50  0001 C CNN
+F 3 "" H 14700 5050 50  0001 C CNN
+	1    14700 5050
 	1    0    0    -1
 $EndComp
@@
 Wire Wire Line
 	3500 1500 3850 1500
+NoConn ~ 14600 4850
+Wire Wire Line
+	1000 7550 1000 7800
+NoConn ~ 900  7550
 $EndSCHEMATC

Commit message: Rev C: Wire in missing I2C bus. Reorder LEDs. Move power rail to avoid colliding with status LEDs.
Parts:
- removed J2: 7SEG_DEBUG, Pin_Headers:Pin_Header_Straight_1x04_Pitch2.54mm, symbol Connector:Conn_01x04_Female
Connections:
- wire segments 140 -> 134
Changed lines of the file:
@@
 NoConn ~ 4650 2000
 NoConn ~ 4650 2100
-$Comp
-L Connector:Conn_01x04_Female J2
-U 1 1 59EEB3FD
-P 2350 1800
-F 0 "J2" H 2350 2000 50  0000 C CNN
-F 1 "7SEG_DEBUG" H 2350 1500 50  0000 C CNN
-F 2 "Pin_Headers:Pin_Header_Straight_1x04_Pitch2.54mm" H 2350 1800 50  0001 C CNN
-F 3 "https://cdn.harwin.com/pdfs/Harwin_Product_Catalog_page_208.pdf" H 2350 1800 50  0001 C CNN
-F 4 "952-2265-ND" H 2350 1800 60  0001 C CNN "S1PN"
-F 5 "https://www.digikey.com/product-detail/en/harwin-inc/M20-9990445/952-2265-ND/3728229" H 2350 1800 60  0001 C CNN "S1PL"
-F 6 "Harwin Inc." H 2350 1800 60  0001 C CNN "MFN"
-F 7 "M20-9990445" H 2350 1800 60  0001 C CNN "MFP"
-	1    2350 1800
-	-1   0    0    1
-$EndComp
 Wire Wire Line
 	4650 1400 9950 1400
@@
 	4200 3000 4200 3200
 Wire Wire Line
-	2100 1400 2650 1400
-Wire Wire Line
 	2550 1700 2750 1700
 Wire Wire Line
@@
 Wire Wire Line
 	2100 1200 2100 1400
-Wire Wire Line
-	2100 3200 2650 3200
 Connection ~ 4200 3200
 Connection ~ 2100 1400
@@
 Wire Wire Line
 	2550 1800 2950 1800
-Wire Wire Line
-	2650 1400 2650 1600
-Wire Wire Line
-	2650 1600 2550 1600
-Connection ~ 2650 1400
-Wire Wire Line
-	2550 1900 2650 1900
-Wire Wire Line
-	2650 1900 2650 3200
-Connection ~ 2650 3200
 Text Notes 14650 13150 0    60   ~ 0
 A
@@
 	2100 1400 2100 1950
 Wire Wire Line
-	2650 3200 4200 3200
-Wire Wire Line
 	2750 1700 3850 1700
 Wire Wire Line
@@
 Text Label 4600 7550 0    50   ~ 0
 7SEG_SDA
-Text Label 2350 1700 2    50   ~ 0
+Text Label 2550 1700 2    50   ~ 0
 7SEG_SDA
-Text Label 2350 1800 2    50   ~ 0
+Text Label 2550 1800 2    50   ~ 0
 7SEG_SCL
 $Comp
@@
 	1    0    0    -1
 $EndComp
-Wire Wire Line
-	2650 1400 3000 1400
 Wire Wire Line
 	3000 1500 3000 1400
@@
 	1000 7550 1000 7800
 NoConn ~ 900  7550
+Wire Wire Line
+	2100 3200 4200 3200
+Wire Wire Line
+	2100 1400 3000 1400
 $EndSCHEMATC
