File: keebee/hardware/keebee/keebee.sch (KiCad schematic (older format))
At the start: 11 parts, among them J1 USB_B_Micro, J2 Conn_ARM_JTAG_SWD_10, U1 LM1117-3.3, U2 STM32F042K6Tx

Commit message: Add status LED, layout dip switch and reset switch.
Parts:
- removed SW_LO: SW_SPST, symbol Switch:SW_SPST
- added D41: LED, symbol Device:LED
- added R1: 300, symbol Device:R
- added SW40: SW_SPST, symbol Switch:SW_SPST
- added SW_LAYOUT: SW_DIP_x02, symbol Switch:SW_DIP_x02
Connections:
- wire segments 88 -> 98
- no-connect marks 6 -> 3
Changed lines of the file:
@@
 Wire Wire Line
 	4700 3400 5000 3400
-NoConn ~ 5000 2500
-NoConn ~ 5000 3000
-NoConn ~ 5000 3100
 Text Label 4700 3300 0    50   ~ 0
 COL8
@@
 Wire Wire Line
 	5000 4000 4400 4000
-$Comp
-L Switch:SW_SPST SW_LO
-U 1 1 5D241928
-P 4200 4000
-F 0 "SW_LO" H 4200 4235 50  0000 C CNN
-F 1 "SW_SPST" H 4200 4144 50  0000 C CNN
-F 2 "" H 4200 4000 50  0001 C CNN
-F 3 "" H 4200 4000 50  0001 C CNN
-	1    4200 4000
-	1    0    0    -1
-$EndComp
-Wire Wire Line
-	4000 4000 3850 4000
-Wire Wire Line
-	3850 4000 3850 4250
-$Comp
-L power:GND #PWR?
-U 1 1 5D244BDB
-P 3850 4250
-F 0 "#PWR?" H 3850 4000 50  0001 C CNN
-F 1 "GND" H 3855 4077 50  0000 C CNN
-F 2 "" H 3850 4250 50  0001 C CNN
-F 3 "" H 3850 4250 50  0001 C CNN
-	1    3850 4250
-	1    0    0    -1
-$EndComp
+Wire Wire Line
+	5000 2500 4500 2500
+$Comp
+L Switch:SW_SPST SW40
+U 1 1 5D247DE4
+P 4300 2500
+F 0 "SW40" H 4300 2735 50  0000 C CNN
+F 1 "SW_SPST" H 4300 2644 50  0000 C CNN
+F 2 "" H 4300 2500 50  0001 C CNN
+F 3 "" H 4300 2500 50  0001 C CNN
+	1    4300 2500
+	1    0    0    -1
+$EndComp
+Wire Wire Line
+	4100 2500 3950 2500
+Wire Wire Line
+	3950 2500 3950 2750
+$Comp
+L power:GND #PWR03
+U 1 1 5D24AD85
+P 3950 2750
+F 0 "#PWR03" H 3950 2500 50  0001 C CNN
+F 1 "GND" H 3955 2577 50  0000 C CNN
+F 2 "" H 3950 2750 50  0001 C CNN
+F 3 "" H 3950 2750 50  0001 C CNN
+	1    3950 2750
+	1    0    0    -1
+$EndComp
+$Comp
+L Device:R R1
+U 1 1 5D24AFA8
+P 4400 4300
+F 0 "R1" H 4470 4346 50  0000 L CNN
+F 1 "300" H 4470 4255 50  0000 L CNN
+F 2 "" V 4330 4300 50  0001 C CNN
+F 3 "~" H 4400 4300 50  0001 C CNN
+	1    4400 4300
+	1    0    0    -1
+$EndComp
+$Comp
+L power:GND #PWR05
+U 1 1 5D250D48
+P 4400 5050
+F 0 "#PWR05" H 4400 4800 50  0001 C CNN
+F 1 "GND" H 4405 4877 50  0000 C CNN
+F 2 "" H 4400 5050 50  0001 C CNN
+F 3 "" H 4400 5050 50  0001 C CNN
+	1    4400 5050
+	1    0    0    -1
+$EndComp
+Wire Wire Line
+	4400 4000 4400 4150
+$Comp
+L Device:LED D41
+U 1 1 5D253E02
+P 4400 4650
+F 0 "D41" V 4438 4533 50  0000 R CNN
+F 1 "LED" V 4347 4533 50  0000 R CNN
+F 2 "" H 4400 4650 50  0001 C CNN
+F 3 "~" H 4400 4650 50  0001 C CNN
+	1    4400 4650
+	0    -1   -1   0
+$EndComp
+Wire Wire Line
+	4400 4450 4400 4500
+Wire Wire Line
+	4400 4800 4400 5050
+$Comp
+L Switch:SW_DIP_x02 SW_LAYOUT
+U 1 1 5D259D35
+P 4500 3100
+F 0 "SW_LAYOUT" H 4500 3467 50  0000 C CNN
+F 1 "SW_DIP_x02" H 4500 3376 50  0000 C CNN
+F 2 "" H 4500 3100 50  0001 C CNN
+F 3 "" H 4500 3100 50  0001 C CNN
+	1    4500 3100
+	1    0    0    -1
+$EndComp
+Wire Wire Line
+	5000 3000 4800 3000
+Wire Wire Line
+	5000 3100 4800 3100
+Wire Wire Line
+	4200 3100 4100 3100
+Wire Wire Line
+	4100 3100 4100 3400
+$Comp
+L power:GND #PWR04
+U 1 1 5D26310C
+P 4100 3400
+F 0 "#PWR04" H 4100 3150 50  0001 C CNN
+F 1 "GND" H 4105 3227 50  0000 C CNN
+F 2 "" H 4100 3400 50  0001 C CNN
+F 3 "" H 4100 3400 50  0001 C CNN
+	1    4100 3400
+	1    0    0    -1
+$EndComp
+Wire Wire Line
+	4200 3000 4100 3000
+Wire Wire Line
+	4100 3000 4100 3100
+Connection ~ 4100 3100
 $EndSCHEMATC

Commit message: Label status led
Parts:
- D41: value LED -> STATUS_LED
Changed lines of the file:
@@
 P 4400 4650
 F 0 "D41" V 4438 4533 50  0000 R CNN
-F 1 "LED" V 4347 4533 50  0000 R CNN
+F 1 "STATUS_LED" V 4347 4533 50  0000 R CNN
 F 2 "" H 4400 4650 50  0001 C CNN
 F 3 "~" H 4400 4650 50  0001 C CNN

Commit message: Relabel components
Parts:
- R1: footprint (none) -> Resistors_SMD:R_0805_HandSoldering
- R2: renamed from R300; value R -> 300
- SW40: value SW_SPST -> SW_RST
- renumbered SW_LAYOUT to SW_LAYOUT1
Changed lines of the file:
@@
 $EndComp
 $Comp
-L Device:R R300
+L Device:R R2
 U 1 1 5B7FDFA5
 P 4350 1100
-F 0 "R300" H 4420 1146 50  0000 L CNN
-F 1 "R" H 4420 1055 50  0000 L CNN
+F 0 "R2" H 4420 1146 50  0000 L CNN
+F 1 "300" H 4420 1055 50  0000 L CNN
 F 2 "Resistors_SMD:R_0805_HandSoldering" V 4280 1100 50  0001 C CNN
 F 3 "~" H 4350 1100 50  0001 C CNN
@@
 P 4300 2500
 F 0 "SW40" H 4300 2735 50  0000 C CNN
-F 1 "SW_SPST" H 4300 2644 50  0000 C CNN
+F 1 "SW_RST" H 4300 2644 50  0000 C CNN
 F 2 "" H 4300 2500 50  0001 C CNN
 F 3 "" H 4300 2500 50  0001 C CNN
@@
 F 0 "R1" H 4470 4346 50  0000 L CNN
 F 1 "300" H 4470 4255 50  0000 L CNN
-F 2 "" V 4330 4300 50  0001 C CNN
+F 2 "Resistors_SMD:R_0805_HandSoldering" V 4330 4300 50  0001 C CNN
 F 3 "~" H 4400 4300 50  0001 C CNN
 	1    4400 4300
@@
 	4400 4800 4400 5050
 $Comp
-L Switch:SW_DIP_x02 SW_LAYOUT
+L Switch:SW_DIP_x02 SW_LAYOUT1
 U 1 1 5D259D35
 P 4500 3100
-F 0 "SW_LAYOUT" H 4500 3467 50  0000 C CNN
+F 0 "SW_LAYOUT1" H 4500 3467 50  0000 C CNN
 F 1 "SW_DIP_x02" H 4500 3376 50  0000 C CNN
 F 2 "" H 4500 3100 50  0001 C CNN

Commit message: Add boot selection switch.
Parts:
- added R3: 10K, symbol Device:R
- added SW_BOOT1: SW_SPST, symbol Switch:SW_SPST
Connections:
- wire segments 98 -> 103
Other:
- moved on the sheet: D41, R1
Changed lines of the file:
@@
 EESchema Schematic File Version 4
+LIBS:keebee-cache
 EELAYER 26 0
 EELAYER END
@@
 SWDIO
 Wire Wire Line
-	5000 4000 4400 4000
-Wire Wire Line
 	5000 2500 4500 2500
 $Comp
@@
 L Device:R R1
 U 1 1 5D24AFA8
-P 4400 4300
-F 0 "R1" H 4470 4346 50  0000 L CNN
-F 1 "300" H 4470 4255 50  0000 L CNN
-F 2 "Resistors_SMD:R_0805_HandSoldering" V 4330 4300 50  0001 C CNN
-F 3 "~" H 4400 4300 50  0001 C CNN
-	1    4400 4300
+P 3600 4300
+F 0 "R1" H 3670 4346 50  0000 L CNN
+F 1 "300" H 3670 4255 50  0000 L CNN
+F 2 "Resistors_SMD:R_0805_HandSoldering" V 3530 4300 50  0001 C CNN
+F 3 "~" H 3600 4300 50  0001 C CNN
+	1    3600 4300
 	1    0    0    -1
 $EndComp
@@
 L power:GND #PWR05
 U 1 1 5D250D48
-P 4400 5050
-F 0 "#PWR05" H 4400 4800 50  0001 C CNN
-F 1 "GND" H 4405 4877 50  0000 C CNN
-F 2 "" H 4400 5050 50  0001 C CNN
-F 3 "" H 4400 5050 50  0001 C CNN
-	1    4400 5050
-	1    0    0    -1
-$EndComp
-Wire Wire Line
-	4400 4000 4400 4150
+P 3600 4900
+F 0 "#PWR05" H 3600 4650 50  0001 C CNN
+F 1 "GND" H 3605 4727 50  0000 C CNN
+F 2 "" H 3600 4900 50  0001 C CNN
+F 3 "" H 3600 4900 50  0001 C CNN
+	1    3600 4900
+	1    0    0    -1
+$EndComp
 $Comp
 L Device:LED D41
 U 1 1 5D253E02
-P 4400 4650
-F 0 "D41" V 4438 4533 50  0000 R CNN
-F 1 "STATUS_LED" V 4347 4533 50  0000 R CNN
-F 2 "" H 4400 4650 50  0001 C CNN
-F 3 "~" H 4400 4650 50  0001 C CNN
-	1    4400 4650
+P 3600 4650
+F 0 "D41" V 3638 4533 50  0000 R CNN
+F 1 "STATUS_LED" V 3547 4533 50  0000 R CNN
+F 2 "" H 3600 4650 50  0001 C CNN
+F 3 "~" H 3600 4650 50  0001 C CNN
+	1    3600 4650
 	0    -1   -1   0
 $EndComp
-Wire Wire Line
-	4400 4450 4400 4500
-Wire Wire Line
-	4400 4800 4400 5050
 $Comp
 L Switch:SW_DIP_x02 SW_LAYOUT1
@@
 	4100 3000 4100 3100
 Connection ~ 4100 3100
+$Comp
+L Device:R R3
+U 1 1 5D26BAFC
+P 4300 4300
+F 0 "R3" H 4370 4346 50  0000 L CNN
+F 1 "10K" H 4370 4255 50  0000 L CNN
+F 2 "" V 4230 4300 50  0001 C CNN
+F 3 "~" H 4300 4300 50  0001 C CNN
+	1    4300 4300
+	1    0    0    -1
+$EndComp
+$Comp
+L power:GND #PWR06
+U 1 1 5D26BB92
+P 4300 4550
+F 0 "#PWR06" H 4300 4300 50  0001 C CNN
+F 1 "GND" H 4305 4377 50  0000 C CNN
+F 2 "" H 4300 4550 50  0001 C CNN
+F 3 "" H 4300 4550 50  0001 C CNN
+	1    4300 4550
+	1    0    0    -1
+$EndComp
+Wire Wire Line
+	3600 4000 3600 4150
+Wire Wire Line
+	3600 4450 3600 4500
+Wire Wire Line
+	3600 4800 3600 4900
+Wire Wire Line
+	4300 4450 4300 4550
+Wire Wire Line
+	4300 4150 4300 4000
+Connection ~ 4300 4000
+Wire Wire Line
+	4300 4000 4450 4000
+$Comp
+L Switch:SW_SPST SW_BOOT1
+U 1 1 5D28D80C
+P 4450 3650
+F 0 "SW_BOOT1" V 4500 3250 50  0000 L CNN
+F 1 "SW_SPST" V 4600 3250 50  0000 L CNN
+F 2 "" H 4450 3650 50  0001 C CNN
+F 3 "" H 4450 3650 50  0001 C CNN
+	1    4450 3650
+	0    1    1    0
+$EndComp
+$Comp
+L power:+3.3V #PWR07
+U 1 1 5D290FE4
+P 4450 3450
+F 0 "#PWR07" H 4450 3300 50  0001 C CNN
+F 1 "+3.3V" H 4465 3623 50  0000 C CNN
+F 2 "" H 4450 3450 50  0001 C CNN
+F 3 "" H 4450 3450 50  0001 C CNN
+	1    4450 3450
+	1    0    0    -1
+$EndComp
+Wire Wire Line
+	4450 3850 4450 4000
+Connection ~ 4450 4000
+Wire Wire Line
+	4450 4000 5000 4000
+Wire Wire Line
+	3600 4000 4300 4000
 $EndSCHEMATC

Commit message: Add 0805 footprints.
Parts:
- D41: footprint (none) -> LEDs:LED_0805_HandSoldering
- R3: footprint (none) -> Resistors_SMD:R_0805_HandSoldering
Changed lines of the file:
@@
 F 0 "D41" V 3638 4533 50  0000 R CNN
 F 1 "STATUS_LED" V 3547 4533 50  0000 R CNN
-F 2 "" H 3600 4650 50  0001 C CNN
+F 2 "LEDs:LED_0805_HandSoldering" H 3600 4650 50  0001 C CNN
 F 3 "~" H 3600 4650 50  0001 C CNN
 	1    3600 4650
@@
 F 0 "R3" H 4370 4346 50  0000 L CNN
 F 1 "10K" H 4370 4255 50  0000 L CNN
-F 2 "" V 4230 4300 50  0001 C CNN
+F 2 "Resistors_SMD:R_0805_HandSoldering" V 4230 4300 50  0001 C CNN
 F 3 "~" H 4300 4300 50  0001 C CNN
 	1    4300 4300

Commit message: Add dip switch footprint, and update BOM.
Parts:
- SW_LAYOUT1: footprint (none) -> custom_switches:219-2MSTR
Changed lines of the file:
@@
 F 0 "SW_LAYOUT1" H 4500 3467 50  0000 C CNN
 F 1 "SW_DIP_x02" H 4500 3376 50  0000 C CNN
-F 2 "" H 4500 3100 50  0001 C CNN
+F 2 "custom_switches:219-2MSTR" H 4500 3100 50  0001 C CNN
 F 3 "" H 4500 3100 50  0001 C CNN
 	1    4500 3100

Commit message: Assign B3F footprint to the reset switch.
Parts:
- SW40: footprint (none) -> Buttons_Switches_THT:SW_TH_Tactile_Omron_B3F-10xx
Changed lines of the file:
@@
 F 0 "SW40" H 4300 2735 50  0000 C CNN
 F 1 "SW_RST" H 4300 2644 50  0000 C CNN
-F 2 "" H 4300 2500 50  0001 C CNN
+F 2 "Buttons_Switches_THT:SW_TH_Tactile_Omron_B3F-10xx" H 4300 2500 50  0001 C CNN
 F 3 "" H 4300 2500 50  0001 C CNN
 	1    4300 2500
