File: keebee/hardware/keebee/keebee.sch (KiCad schematic (older format))
At the start: 16 parts, among them J1 USB_B_Micro, J2 Conn_ARM_JTAG_SWD_10, SW40 SW_RST, U1 LM1117-3.3, U2 STM32F042K6Tx

Commit message: Fixup imported footprint errors.
Parts:
- removed R3: 10K, Resistors_SMD:R_0805_HandSoldering, symbol Device:R
Connections:
- wire segments 103 -> 100
Changed lines of the file:
@@
 	4100 3000 4100 3100
 Connection ~ 4100 3100
-$Comp
-L Device:R R3
-U 1 1 5D26BAFC
-P 4300 4300
-F 0 "R3" H 4370 4346 50  0000 L CNN
-F 1 "10K" H 4370 4255 50  0000 L CNN
-F 2 "Resistors_SMD:R_0805_HandSoldering" V 4230 4300 50  0001 C CNN
-F 3 "~" H 4300 4300 50  0001 C CNN
-	1    4300 4300
-	1    0    0    -1
-$EndComp
-$Comp
-L power:GND #PWR06
-U 1 1 5D26BB92
-P 4300 4550
-F 0 "#PWR06" H 4300 4300 50  0001 C CNN
-F 1 "GND" H 4305 4377 50  0000 C CNN
-F 2 "" H 4300 4550 50  0001 C CNN
-F 3 "" H 4300 4550 50  0001 C CNN
-	1    4300 4550
-	1    0    0    -1
-$EndComp
 Wire Wire Line
 	3600 4000 3600 4150
@@
 Wire Wire Line
 	3600 4800 3600 4900
-Wire Wire Line
-	4300 4450 4300 4550
-Wire Wire Line
-	4300 4150 4300 4000
-Connection ~ 4300 4000
 $Comp
 L Switch:SW_SPST SW_BOOT0
@@
 	3600 4000 3900 4000
 Wire Wire Line
-	4300 4000 5000 4000
-Wire Wire Line
 	3900 3900 3900 4000
 Connection ~ 3900 4000
 Wire Wire Line
-	3900 4000 4300 4000
+	3900 4000 5000 4000
 $EndSCHEMATC

Commit message: Route more trackes.
Parts:
- J2: footprint Connector_PinHeader_1.27mm:PinHeader_2x05_P1.27mm_Vertical_SMD -> Pin_Headers:Pin_Header_Straight_2x05_Pitch1.27mm_SMD
- U2: footprint Package_QFP:LQFP-32_7x7mm_P0.8mm -> Housings_QFP:LQFP-32_7x7mm_Pitch0.8mm
Connections:
- no-connect marks 3 -> 5
Changed lines of the file:
@@
 F 0 "U2" H 5500 2114 50  0000 C CNN
 F 1 "STM32F042K6Tx" H 5500 2023 50  0000 C CNN
-F 2 "Package_QFP:LQFP-32_7x7mm_P0.8mm" H 5100 2300 50  0001 R CNN
+F 2 "Housings_QFP:LQFP-32_7x7mm_Pitch0.8mm" H 5100 2300 50  0001 R CNN
 F 3 "http://www.st.com/st-web-ui/static/active/en/resource/technical/document/datasheet/DM00105814.pdf" H 5500 3200 50  0001 C CNN
 	1    5500 3200
@@
 F 0 "J2" H 1910 5896 50  0000 R CNN
 F 1 "Conn_ARM_JTAG_SWD_10" H 1910 5805 50  0000 R CNN
-F 2 "Connector_PinHeader_1.27mm:PinHeader_2x05_P1.27mm_Vertical_SMD" H 2400 5300 50  0001 L TNN
+F 2 "Pin_Headers:Pin_Header_Straight_2x05_Pitch1.27mm_SMD" H 2400 5300 50  0001 L TNN
 F 3 "http://infocenter.arm.com/help/topic/com.arm.doc.faqs/attached/13634/cortex_debug_connectors.pdf" V 2000 4600 50  0001 C CNN
 	1    2350 5850
@@
 Wire Wire Line
 	3900 4000 5000 4000
+NoConn ~ 2850 5950
+NoConn ~ 2850 6050
 $EndSCHEMATC

Commit message: Remove dip switch, fix button pinout. Rev. 2.
Parts:
- removed SW_LAYOUT1: SW_DIP_x02, custom_switches:219-2MSTR, symbol Switch:SW_DIP_x02
- SW40, SW_BOOT0: footprint Buttons_Switches_THT:SW_TH_Tactile_Omron_B3F-10xx -> Button_Switch_THT:SW_PUSH_6mm
Connections:
- wire segments 100 -> 94
- no-connect marks 5 -> 7
Changed lines of the file:
@@
 Comment4 ""
 $EndDescr
-$Comp
-L MCU_ST_STM32F0:STM32F042K6Tx U2
-U 1 1 5B304C68
-P 5500 3200
-F 0 "U2" H 5500 2114 50  0000 C CNN
-F 1 "STM32F042K6Tx" H 5500 2023 50  0000 C CNN
-F 2 "Housings_QFP:LQFP-32_7x7mm_Pitch0.8mm" H 5100 2300 50  0001 R CNN
-F 3 "http://www.st.com/st-web-ui/static/active/en/resource/technical/document/datasheet/DM00105814.pdf" H 5500 3200 50  0001 C CNN
-	1    5500 3200
-	1    0    0    -1
-$EndComp
 Wire Wire Line
 	5400 4200 5400 4300
@@
 F 0 "SW40" H 4300 2735 50  0000 C CNN
 F 1 "SW_RST" H 4300 2644 50  0000 C CNN
-F 2 "Buttons_Switches_THT:SW_TH_Tactile_Omron_B3F-10xx" H 4300 2500 50  0001 C CNN
+F 2 "Button_Switch_THT:SW_PUSH_6mm" H 4300 2500 50  0001 C CNN
 F 3 "" H 4300 2500 50  0001 C CNN
 	1    4300 2500
@@
 	0    -1   -1   0
 $EndComp
-$Comp
-L Switch:SW_DIP_x02 SW_LAYOUT1
-U 1 1 5D259D35
-P 4500 3100
-F 0 "SW_LAYOUT1" H 4500 3467 50  0000 C CNN
-F 1 "SW_DIP_x02" H 4500 3376 50  0000 C CNN
-F 2 "custom_switches:219-2MSTR" H 4500 3100 50  0001 C CNN
-F 3 "" H 4500 3100 50  0001 C CNN
-	1    4500 3100
-	1    0    0    -1
-$EndComp
-Wire Wire Line
-	5000 3000 4800 3000
-Wire Wire Line
-	5000 3100 4800 3100
-Wire Wire Line
-	4200 3100 4100 3100
-Wire Wire Line
-	4100 3100 4100 3400
-$Comp
-L power:GND #PWR04
-U 1 1 5D26310C
-P 4100 3400
-F 0 "#PWR04" H 4100 3150 50  0001 C CNN
-F 1 "GND" H 4105 3227 50  0000 C CNN
-F 2 "" H 4100 3400 50  0001 C CNN
-F 3 "" H 4100 3400 50  0001 C CNN
-	1    4100 3400
-	1    0    0    -1
-$EndComp
-Wire Wire Line
-	4200 3000 4100 3000
-Wire Wire Line
-	4100 3000 4100 3100
-Connection ~ 4100 3100
 Wire Wire Line
 	3600 4000 3600 4150
@@
 F 0 "SW_BOOT0" V 3950 3300 50  0000 L CNN
 F 1 "SW_SPST" V 4050 3300 50  0000 L CNN
-F 2 "Buttons_Switches_THT:SW_TH_Tactile_Omron_B3F-10xx" H 3900 3700 50  0001 C CNN
+F 2 "Button_Switch_THT:SW_PUSH_6mm" H 3900 3700 50  0001 C CNN
 F 3 "" H 3900 3700 50  0001 C CNN
 	1    3900 3700
@@
 NoConn ~ 2850 5950
 NoConn ~ 2850 6050
+$Comp
+L MCU_ST_STM32F0:STM32F042K6Tx U2
+U 1 1 5B304C68
+P 5500 3200
+F 0 "U2" H 5500 2114 50  0000 C CNN
+F 1 "STM32F042K6Tx" H 5500 2023 50  0000 C CNN
+F 2 "Housings_QFP:LQFP-32_7x7mm_Pitch0.8mm" H 5100 2300 50  0001 R CNN
+F 3 "http://www.st.com/st-web-ui/static/active/en/resource/technical/document/datasheet/DM00105814.pdf" H 5500 3200 50  0001 C CNN
+	1    5500 3200
+	1    0    0    -1
+$EndComp
+NoConn ~ 5000 3000
+NoConn ~ 5000 3100
 $EndSCHEMATC
