File: keebee/hardware/keebee/keebee.kicad_pcb (KiCad board)
At the start: 2 copper layers, 275 x 103 mm, 160 parts, among them J1 USB_B_Micro, J2 Conn_ARM_JTAG_SWD_10, SW1 SW_SPST, SW10 SW_SPST, SW11 SW_SPST, SW12 SW_SPST, SW13 SW_SPST, SW14 SW_SPST, SW15 SW_SPST, SW16 SW_SPST, SW17 SW_SPST, SW18 SW_SPST, SW19 SW_SPST, SW2 SW_SPST, SW20 SW_SPST, SW21 SW_SPST, SW22 SW_SPST, SW23 SW_SPST, SW24 SW_SPST, SW25 SW_SPST, SW26 SW_SPST, SW27 SW_SPST, SW28 SW_SPST, SW29 SW_SPST, SW3 SW_SPST, SW30 SW_SPST, SW31 SW_SPST, SW32 SW_SPST, SW33 SW_SPST, SW34 SW_SPST, SW35 SW_SPST, SW36 SW_SPST, SW37 SW_SPST, SW38 SW_SPST, SW39 SW_SPST, SW4 SW_SPST, SW41 SW_SPST, SW42 SW_SPST, SW43 SW_SPST, SW44 SW_SPST, SW45 SW_SPST, SW46 SW_SPST, SW47 SW_SPST, SW48 SW_SPST, SW49 SW_SPST, SW5 SW_SPST, SW50 SW_SPST, SW51 SW_SPST, SW52 SW_SPST, SW53 SW_SPST, SW54 SW_SPST, SW55 SW_SPST, SW56 SW_SPST, SW57 SW_SPST, SW58 SW_SPST, SW59 SW_SPST, SW6 SW_SPST, SW60 SW_SPST, SW61 SW_SPST, SW62 SW_SPST, SW63 SW_SPST, SW64 SW_SPST, SW65 SW_SPST, SW66 SW_SPST, SW67 SW_SPST, SW68 SW_SPST, SW69 SW_SPST, SW7 SW_SPST, SW70 SW_SPST, SW8 SW_SPST, SW9 SW_SPST, U1 LM1117-3.3, U2 STM32F042K6Tx

Commit message: Move Keebee logo to the back.
Parts:
- G***: moved to B.Cu
- moved G*** 208.5 mm to (59.4, 93.5), turned to 180 degrees

Commit message: Remove dip switch, fix button pinout. Rev. 2.
Parts:
- removed SW_LAYOUT1: SW_DIP_x02, custom_switches:219-2MSTR
- removed SW_RST: SW_RST, Buttons_Switches_THT:SW_TH_Tactile_Omron_B3F-10xx
- added SW40: SW_RST, Button_Switch_THT:SW_PUSH_6mm, B.Cu at (140.3, 63.2)
- SW_BOOT0: footprint Buttons_Switches_THT:SW_TH_Tactile_Omron_B3F-10xx -> Button_Switch_THT:SW_PUSH_6mm
- moved J2 2.67 mm to (155.6, 60.5)
Routing:
- net Net-(U2-Pad3): track 57.6 -> 0.00 mm, vias 2 -> 0
- net Net-(U2-Pad2): track 47.4 -> 0.00 mm, vias 2 -> 0
- net GND: track 79.7 -> 112.1 mm, vias 15 -> 17
- net Net-(SW40-Pad2): track 55.4 -> 78.2 mm, vias 4 -> 6
- net Net-(R1-Pad1): track 80.3 -> 93.1 mm
- net +3V3: track 415.1 -> 424.0 mm
- net /SWCLK: track 56.3 -> 50.6 mm
- net /SWDIO: track 54.5 -> 57.1 mm
- net Net-(J2-Pad8): track 0.00 -> 0.83 mm
- net Net-(J2-Pad6): track 0.00 -> 0.83 mm
- net Net-(J1-Pad2): track 180.5 -> 181.2 mm
Other:
- board text added: "KeeBee rev. 2"
- board text removed: "KeeBee rev. 1"
