File: ww/hardware/ww/ww.sch (KiCad schematic (older format))
At the start: 49 parts, among them J1 USB_B, J2 Conn_ARM_JTAG_SWD_10, SW1 BTN0, SW2 BTN1, U1 MCP73812T-420I-OT, U10 APA102, U11 APA102, U12 APA102, U13 APA102, U14 APA102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

Commit message: Use side-angled SMT JST battery connector
Parts:
- BT1: footprint Connectors_JST:JST_PH_B2B-PH-K_02x2.00mm_Straight -> Connectors_JST:JST_PH_S2B-PH-SM4-TB_02x2.00mm_Angled
Changed lines of the file:
@@
 F 0 "BT1" H 3618 2396 50  0000 L CNN
 F 1 "Battery_Cell" H 3618 2305 50  0000 L CNN
-F 2 "Connectors_JST:JST_PH_B2B-PH-K_02x2.00mm_Straight" V 3500 2360 50  0001 C CNN
+F 2 "Connectors_JST:JST_PH_S2B-PH-SM4-TB_02x2.00mm_Angled" V 3500 2360 50  0001 C CNN
 F 3 "~" V 3500 2360 50  0001 C CNN
 	1    3500 2300
