File: oxidized_flash/hardware/oxidized_flash/oxidized_flash.sch (KiCad schematic (older format))
At the start: 19 parts, among them J1 USB_A, J2 Conn_ARM_JTAG_SWD_10, U1 LM1117-3.3, U2 ATSAMD51G18A-MU, U3 MT25QL

Commit message: Add reset pin to SWD header
Connections:
- wire segments 83 -> 84
- no-connect marks 8 -> 7
Changed lines of the file:
@@
 	950  1200 1300 1200
 NoConn ~ 4400 4750
-Wire Wire Line
-	3450 5050 3450 5300
-NoConn ~ 2650 3200
-$Comp
-L ATSAMD:ATSAMD51G18A-MU U2
-U 1 1 5E0421D4
-P 3600 3350
-F 0 "U2" H 3525 5281 50  0000 C CNN
-F 1 "ATSAMD51G18A-MU" H 3525 5190 50  0000 C CNN
-F 2 "Housings_DFN_QFN:QFN-48-1EP_7x7mm_Pitch0.5mm" H 3600 3350 50  0001 C CNN
-F 3 "" H 3600 3350 50  0001 C CNN
-	1    3600 3350
-	1    0    0    -1
-$EndComp
 $Comp
 L custom_ic:MT25QL U3
@@
 Wire Wire Line
 	2000 4100 2650 4100
+Wire Wire Line
+	3450 5050 3450 5300
+$Comp
+L ATSAMD:ATSAMD51G18A-MU U2
+U 1 1 5E0421D4
+P 3600 3350
+F 0 "U2" H 3525 5281 50  0000 C CNN
+F 1 "ATSAMD51G18A-MU" H 3525 5190 50  0000 C CNN
+F 2 "Housings_DFN_QFN:QFN-48-1EP_7x7mm_Pitch0.5mm" H 3600 3350 50  0001 C CNN
+F 3 "" H 3600 3350 50  0001 C CNN
+	1    3600 3350
+	1    0    0    -1
+$EndComp
+Wire Wire Line
+	2650 3200 2000 3200
+Text Label 2000 3200 0    50   ~ 0
+SWD_RST
 $EndSCHEMATC

Commit message: Switch 0603 to handsoldering for more room
Parts:
- C1, C4, C5, C6, C7, C8, C9: footprint Capacitors_SMD:C_0603 -> Capacitors_SMD:C_0603_HandSoldering
- D1, D4: footprint LEDs:LED_0603 -> LEDs:LED_0603_HandSoldering
- R1, R8: footprint Resistors_SMD:R_0603 -> Resistors_SMD:R_0603_HandSoldering
Changed lines of the file:
@@
 F 0 "C4" H 4342 1296 50  0000 L CNN
 F 1 "10u" H 4342 1205 50  0000 L CNN
-F 2 "Capacitors_SMD:C_0603" H 4250 1250 50  0001 C CNN
+F 2 "Capacitors_SMD:C_0603_HandSoldering" H 4250 1250 50  0001 C CNN
 F 3 "~" H 4250 1250 50  0001 C CNN
 	1    4250 1250
@@
 F 0 "C5" H 4642 1296 50  0000 L CNN
 F 1 "10u" H 4642 1205 50  0000 L CNN
-F 2 "Capacitors_SMD:C_0603" H 4550 1250 50  0001 C CNN
+F 2 "Capacitors_SMD:C_0603_HandSoldering" H 4550 1250 50  0001 C CNN
 F 3 "~" H 4550 1250 50  0001 C CNN
 	1    4550 1250
@@
 F 0 "C7" H 4942 1296 50  0000 L CNN
 F 1 "10u" H 4942 1205 50  0000 L CNN
-F 2 "Capacitors_SMD:C_0603" H 4850 1250 50  0001 C CNN
+F 2 "Capacitors_SMD:C_0603_HandSoldering" H 4850 1250 50  0001 C CNN
 F 3 "~" H 4850 1250 50  0001 C CNN
 	1    4850 1250
@@
 F 0 "C9" H 5242 1296 50  0000 L CNN
 F 1 "10u" H 5242 1205 50  0000 L CNN
-F 2 "Capacitors_SMD:C_0603" H 5150 1250 50  0001 C CNN
+F 2 "Capacitors_SMD:C_0603_HandSoldering" H 5150 1250 50  0001 C CNN
 F 3 "~" H 5150 1250 50  0001 C CNN
 	1    5150 1250
@@
 F 0 "C8" H 5192 4896 50  0000 L CNN
 F 1 "0.1u" H 5192 4805 50  0000 L CNN
-F 2 "Capacitors_SMD:C_0603" H 5100 4850 50  0001 C CNN
+F 2 "Capacitors_SMD:C_0603_HandSoldering" H 5100 4850 50  0001 C CNN
 F 3 "~" H 5100 4850 50  0001 C CNN
 	1    5100 4850
@@
 F 0 "C6" H 4842 4896 50  0000 L CNN
 F 1 "4.7u" H 4842 4805 50  0000 L CNN
-F 2 "Capacitors_SMD:C_0603" H 4750 4850 50  0001 C CNN
+F 2 "Capacitors_SMD:C_0603_HandSoldering" H 4750 4850 50  0001 C CNN
 F 3 "~" H 4750 4850 50  0001 C CNN
 	1    4750 4850
@@
 F 0 "R1" H 1109 4496 50  0000 L CNN
 F 1 "1k" H 1109 4405 50  0000 L CNN
-F 2 "Resistors_SMD:R_0603" H 1050 4450 50  0001 C CNN
+F 2 "Resistors_SMD:R_0603_HandSoldering" H 1050 4450 50  0001 C CNN
 F 3 "~" H 1050 4450 50  0001 C CNN
 	1    1050 4450
@@
 F 0 "D1" V 1096 4082 50  0000 R CNN
 F 1 "OK_Led" V 1005 4082 50  0000 R CNN
-F 2 "LEDs:LED_0603" V 1050 4150 50  0001 C CNN
+F 2 "LEDs:LED_0603_HandSoldering" V 1050 4150 50  0001 C CNN
 F 3 "~" V 1050 4150 50  0001 C CNN
 	1    1050 4150
@@
 F 0 "D4" V 1596 4082 50  0000 R CNN
 F 1 "PWR_LED" V 1505 4082 50  0000 R CNN
-F 2 "LEDs:LED_0603" V 1550 4150 50  0001 C CNN
+F 2 "LEDs:LED_0603_HandSoldering" V 1550 4150 50  0001 C CNN
 F 3 "~" V 1550 4150 50  0001 C CNN
 	1    1550 4150
@@
 F 0 "R8" H 1609 4496 50  0000 L CNN
 F 1 "1k" H 1609 4405 50  0000 L CNN
-F 2 "Resistors_SMD:R_0603" H 1550 4450 50  0001 C CNN
+F 2 "Resistors_SMD:R_0603_HandSoldering" H 1550 4450 50  0001 C CNN
 F 3 "~" H 1550 4450 50  0001 C CNN
 	1    1550 4450
@@
 F 0 "C1" H 6342 3796 50  0000 L CNN
 F 1 "0.1u" H 6342 3705 50  0000 L CNN
-F 2 "Capacitors_SMD:C_0603" H 6250 3750 50  0001 C CNN
+F 2 "Capacitors_SMD:C_0603_HandSoldering" H 6250 3750 50  0001 C CNN
 F 3 "~" H 6250 3750 50  0001 C CNN
 	1    6250 3750

Commit message: Connect reset lines to the flash memory
Connections:
- wire segments 84 -> 82
- no-connect marks 7 -> 8
Changed lines of the file:
@@
 	1    0    0    -1
 $EndComp
-Wire Wire Line
-	2000 6600 2000 6700
-Wire Wire Line
-	2000 6700 2100 6700
-Wire Wire Line
-	2100 6700 2100 6600
 $Comp
 L power:GND #PWR0101
@@
 	1    0    0    -1
 $EndComp
-Wire Wire Line
-	2100 6700 2100 6800
-Connection ~ 2100 6700
 Text Label 2650 5700 0    50   ~ 0
 SWD_RST
@@
 	950  1200 1300 1200
 NoConn ~ 4400 4750
+Wire Wire Line
+	4400 3600 5200 3600
+Wire Wire Line
+	1900 2600 2650 2600
+Wire Wire Line
+	1900 2700 2650 2700
+Wire Wire Line
+	2450 3400 2650 3400
+Wire Wire Line
+	2000 4200 2650 4200
+Wire Wire Line
+	2450 3500 2650 3500
+Wire Wire Line
+	4400 3700 5200 3700
+Wire Wire Line
+	4400 3800 5200 3800
+Wire Wire Line
+	4400 3900 5200 3900
+Wire Wire Line
+	4400 4000 5200 4000
+Wire Wire Line
+	4400 4100 5200 4100
+$Comp
+L Device:C_Small C1
+U 1 1 5E055AF7
+P 6250 3750
+F 0 "C1" H 6342 3796 50  0000 L CNN
+F 1 "0.1u" H 6342 3705 50  0000 L CNN
+F 2 "Capacitors_SMD:C_0603_HandSoldering" H 6250 3750 50  0001 C CNN
+F 3 "~" H 6250 3750 50  0001 C CNN
+	1    6250 3750
+	1    0    0    -1
+$EndComp
+Wire Wire Line
+	5550 3100 6100 3100
+Wire Wire Line
+	6250 3100 6250 3650
+Wire Wire Line
+	6250 3850 6250 4500
+Wire Wire Line
+	6250 4500 6100 4500
+$Comp
+L power:+3.3V #PWR08
+U 1 1 5E05A40F
+P 6100 2950
+F 0 "#PWR08" H 6100 2800 50  0001 C CNN
+F 1 "+3.3V" H 6115 3123 50  0000 C CNN
+F 2 "" H 6100 2950 50  0001 C CNN
+F 3 "" H 6100 2950 50  0001 C CNN
+	1    6100 2950
+	1    0    0    -1
+$EndComp
+Wire Wire Line
+	6100 3100 6100 2950
+Connection ~ 6100 3100
+Wire Wire Line
+	6100 3100 6250 3100
+$Comp
+L power:GND #PWR09
+U 1 1 5E05E6A1
+P 6100 4650
+F 0 "#PWR09" H 6100 4400 50  0001 C CNN
+F 1 "GND" H 6105 4477 50  0000 C CNN
+F 2 "" H 6100 4650 50  0001 C CNN
+F 3 "" H 6100 4650 50  0001 C CNN
+	1    6100 4650
+	1    0    0    -1
+$EndComp
+Wire Wire Line
+	6100 4500 6100 4650
+Connection ~ 6100 4500
+Wire Wire Line
+	6100 4500 5550 4500
+Wire Wire Line
+	2000 4100 2650 4100
+Wire Wire Line
+	3450 5050 3450 5300
+$Comp
+L ATSAMD:ATSAMD51G18A-MU U2
+U 1 1 5E0421D4
+P 3600 3350
+F 0 "U2" H 3525 5281 50  0000 C CNN
+F 1 "ATSAMD51G18A-MU" H 3525 5190 50  0000 C CNN
+F 2 "Housings_DFN_QFN:QFN-48-1EP_7x7mm_Pitch0.5mm" H 3600 3350 50  0001 C CNN
+F 3 "" H 3600 3350 50  0001 C CNN
+	1    3600 3350
+	1    0    0    -1
+$EndComp
+Wire Wire Line
+	2650 3200 2000 3200
+Text Label 2000 3200 0    50   ~ 0
+SWD_RST
+Wire Wire Line
+	2100 6600 2100 6800
+NoConn ~ 2000 6600
 $Comp
 L custom_ic:MT25QL U3
@@
 	1    0    0    -1
 $EndComp
-Wire Wire Line
-	4400 3600 5200 3600
-Wire Wire Line
-	1900 2600 2650 2600
-Wire Wire Line
-	1900 2700 2650 2700
-Wire Wire Line
-	2450 3400 2650 3400
-Wire Wire Line
-	2000 4200 2650 4200
-Wire Wire Line
-	2450 3500 2650 3500
-Wire Wire Line
-	4400 3700 5200 3700
-Wire Wire Line
-	4400 3800 5200 3800
-Wire Wire Line
-	4400 3900 5200 3900
-Wire Wire Line
-	4400 4000 5200 4000
-Wire Wire Line
-	4400 4100 5200 4100
-$Comp
-L Device:C_Small C1
-U 1 1 5E055AF7
-P 6250 3750
-F 0 "C1" H 6342 3796 50  0000 L CNN
-F 1 "0.1u" H 6342 3705 50  0000 L CNN
-F 2 "Capacitors_SMD:C_0603_HandSoldering" H 6250 3750 50  0001 C CNN
-F 3 "~" H 6250 3750 50  0001 C CNN
-	1    6250 3750
-	1    0    0    -1
-$EndComp
-Wire Wire Line
-	5550 3100 6100 3100
-Wire Wire Line
-	6250 3100 6250 3650
-Wire Wire Line
-	6250 3850 6250 4500
-Wire Wire Line
-	6250 4500 6100 4500
-$Comp
-L power:+3.3V #PWR08
-U 1 1 5E05A40F
-P 6100 2950
-F 0 "#PWR08" H 6100 2800 50  0001 C CNN
-F 1 "+3.3V" H 6115 3123 50  0000 C CNN
-F 2 "" H 6100 2950 50  0001 C CNN
-F 3 "" H 6100 2950 50  0001 C CNN
-	1    6100 2950
-	1    0    0    -1
-$EndComp
-Wire Wire Line
-	6100 3100 6100 2950
-Connection ~ 6100 3100
-Wire Wire Line
-	6100 3100 6250 3100
-$Comp
-L power:GND #PWR09
-U 1 1 5E05E6A1
-P 6100 4650
-F 0 "#PWR09" H 6100 4400 50  0001 C CNN
-F 1 "GND" H 6105 4477 50  0000 C CNN
-F 2 "" H 6100 4650 50  0001 C CNN
-F 3 "" H 6100 4650 50  0001 C CNN
-	1    6100 4650
-	1    0    0    -1
-$EndComp
-Wire Wire Line
-	6100 4500 6100 4650
-Connection ~ 6100 4500
-Wire Wire Line
-	6100 4500 5550 4500
-Wire Wire Line
-	2000 4100 2650 4100
-Wire Wire Line
-	3450 5050 3450 5300
-$Comp
-L ATSAMD:ATSAMD51G18A-MU U2
-U 1 1 5E0421D4
-P 3600 3350
-F 0 "U2" H 3525 5281 50  0000 C CNN
-F 1 "ATSAMD51G18A-MU" H 3525 5190 50  0000 C CNN
-F 2 "Housings_DFN_QFN:QFN-48-1EP_7x7mm_Pitch0.5mm" H 3600 3350 50  0001 C CNN
-F 3 "" H 3600 3350 50  0001 C CNN
-	1    3600 3350
-	1    0    0    -1
-$EndComp
-Wire Wire Line
-	2650 3200 2000 3200
-Text Label 2000 3200 0    50   ~ 0
+Text Label 4800 3450 0    50   ~ 0
 SWD_RST
+Wire Wire Line
+	4800 3450 5200 3450
 $EndSCHEMATC
